File: ShutdownCircuit.sch (KiCad schematic (older format))
At the start: 8 parts, among them K1 IMD_RELAY, K2 IMD_LATCH, K3 BMS_RELAY, Q3 Q_NMOS_DGS, Q4 Q_NMOS_DGS, SW1 SW_Push

Commit message: added noel's revisions
Parts:
- added D? (x2): LED, symbol LED
- added R? (x2): R, symbol R
Connections:
- net labels added: IMD_FLT_12V_LED_H
- wire segments 26 -> 36
Changed lines of the file:
@@
 $EndComp
 $Comp
-L +12V #PWR14
+L +12V #PWR20
 U 1 1 5A022276
-P 2900 2050
-F 0 "#PWR14" H 2900 1900 50  0001 C CNN
-F 1 "+12V" H 2900 2190 50  0000 C CNN
-F 2 "" H 2900 2050 50  0001 C CNN
-F 3 "" H 2900 2050 50  0001 C CNN
-	1    2900 2050
-	1    0    0    -1
-$EndComp
-$Comp
-L +12V #PWR15
+P 2900 2150
+F 0 "#PWR20" H 2900 2000 50  0001 C CNN
+F 1 "+12V" H 2900 2290 50  0000 C CNN
+F 2 "" H 2900 2150 50  0001 C CNN
+F 3 "" H 2900 2150 50  0001 C CNN
+	1    2900 2150
+	1    0    0    -1
+$EndComp
+$Comp
+L +12V #PWR21
 U 1 1 5A02229A
-P 3050 3250
-F 0 "#PWR15" H 3050 3100 50  0001 C CNN
-F 1 "+12V" H 3050 3390 50  0000 C CNN
-F 2 "" H 3050 3250 50  0001 C CNN
-F 3 "" H 3050 3250 50  0001 C CNN
-	1    3050 3250
-	1    0    0    -1
-$EndComp
-$Comp
-L +12V #PWR17
+P 3050 3350
+F 0 "#PWR21" H 3050 3200 50  0001 C CNN
+F 1 "+12V" H 3050 3490 50  0000 C CNN
+F 2 "" H 3050 3350 50  0001 C CNN
+F 3 "" H 3050 3350 50  0001 C CNN
+	1    3050 3350
+	1    0    0    -1
+$EndComp
+$Comp
+L +12V #PWR23
 U 1 1 5A0222EA
 P 5250 2550
-F 0 "#PWR17" H 5250 2400 50  0001 C CNN
+F 0 "#PWR23" H 5250 2400 50  0001 C CNN
 F 1 "+12V" H 5250 2690 50  0000 C CNN
 F 2 "" H 5250 2550 50  0001 C CNN
@@
 $EndComp
 $Comp
-L GND #PWR16
+L GND #PWR22
 U 1 1 5A022431
 P 4850 5250
-F 0 "#PWR16" H 4850 5000 50  0001 C CNN
+F 0 "#PWR22" H 4850 5000 50  0001 C CNN
 F 1 "GND" H 4850 5100 50  0000 C CNN
 F 2 "" H 4850 5250 50  0001 C CNN
@@
 Text HLabel 6200 4850 0    60   Input ~ 0
 BMS_FLT_5V_L
-Text HLabel 6050 2150 2    60   Output ~ 0
+Text HLabel 6050 2050 2    60   Output ~ 0
 SD_CKT_DOWNSTREAM
 $Comp
@@
 $EndComp
 Wire Wire Line
-	4850 5250 4850 5050
+	4850 5050 4850 5250
 Wire Wire Line
 	4850 2550 4850 4650
@@
 	3850 4250 4150 4250
 Wire Wire Line
-	3850 2550 3850 4250
+	3850 2550 3850 4550
 Wire Wire Line
 	3850 2550 4000 2550
 Wire Wire Line
-	4600 3350 4600 2900
-Wire Wire Line
-	4600 2900 3850 2900
+	3850 2900 4750 2900
 Connection ~ 3850 2900
 Wire Wire Line
-	3050 3250 4000 3250
-Wire Wire Line
-	3250 3000 3250 3250
-Connection ~ 3250 3250
+	3050 3350 4000 3350
+Wire Wire Line
+	3250 3000 3250 3350
+Connection ~ 3250 3350
 Wire Wire Line
 	3650 3000 3850 3000
 Connection ~ 3850 3000
 Wire Wire Line
-	2900 2050 4000 2050
-Wire Wire Line
-	4600 2150 4600 2050
-Wire Wire Line
-	4600 2050 5450 2050
-Wire Wire Line
 	6500 5050 6500 5200
 Wire Wire Line
@@
 Connection ~ 4850 5200
 Wire Wire Line
-	6500 4650 6500 2550
-Wire Wire Line
-	6500 2550 6050 2550
-Wire Wire Line
-	5450 2550 5250 2550
+	6500 2550 6500 4650
+Wire Wire Line
+	6050 2550 6500 2550
+Wire Wire Line
+	5250 2550 5450 2550
 Wire Wire Line
 	4600 3750 4850 3750
@@
 Connection ~ 3850 3750
 Wire Wire Line
-	5900 2950 6150 2950
-Wire Wire Line
-	6150 2950 6150 2550
-Connection ~ 6150 2550
+	5900 2950 6350 2950
 Wire Wire Line
 	5600 2950 5350 2950
-Wire Wire Line
-	5350 2950 5350 2550
-Connection ~ 5350 2550
 $Comp
 L G5Q-1 K1
 U 1 1 5A023295
-P 4500 2550
-F 0 "K1" H 5150 2900 50  0000 L CNN
-F 1 "IMD_RELAY" H 5150 2800 50  0000 L CNN
-F 2 "Relays_THT:Relay_SPDT_OMRON-G5LE-1" H 5150 2700 50  0001 L CNN
-F 3 "" H 5150 2400 50  0001 L CNN
-	1    4500 2550
-	0    -1   -1   0
+P 4100 2550
+F 0 "K1" H 4750 2900 50  0000 L CNN
+F 1 "IMD_RELAY" H 4750 2800 50  0000 L CNN
+F 2 "Relays_THT:Relay_SPDT_OMRON-G5LE-1" H 4750 2700 50  0001 L CNN
+F 3 "" H 4750 2400 50  0001 L CNN
+	1    4100 2550
+	0    1    -1   0
 $EndComp
 $Comp
 L G5Q-1 K2
 U 1 1 5A0234D4
-P 4500 3750
-F 0 "K2" H 5150 4100 50  0000 L CNN
-F 1 "IMD_LATCH" H 5150 4000 50  0000 L CNN
-F 2 "Relays_THT:Relay_SPDT_OMRON-G5LE-1" H 5150 3900 50  0001 L CNN
-F 3 "" H 5150 3600 50  0001 L CNN
-	1    4500 3750
-	0    -1   -1   0
+P 4100 3750
+F 0 "K2" H 4750 4100 50  0000 L CNN
+F 1 "IMD_LATCH" H 4750 4000 50  0000 L CNN
+F 2 "Relays_THT:Relay_SPDT_OMRON-G5LE-1" H 4750 3900 50  0001 L CNN
+F 3 "" H 4750 3600 50  0001 L CNN
+	1    4100 3750
+	0    1    -1   0
 $EndComp
 $Comp
 L G5Q-1 K3
 U 1 1 5A023534
-P 5950 2550
-F 0 "K3" H 6600 2900 50  0000 L CNN
-F 1 "BMS_RELAY" H 6600 2800 50  0000 L CNN
-F 2 "Relays_THT:Relay_SPDT_OMRON-G5LE-1" H 6600 2700 50  0001 L CNN
-F 3 "" H 6600 2400 50  0001 L CNN
-	1    5950 2550
-	0    -1   -1   0
-$EndComp
+P 5550 2550
+F 0 "K3" H 6200 2900 50  0000 L CNN
+F 1 "BMS_RELAY" H 6200 2800 50  0000 L CNN
+F 2 "Relays_THT:Relay_SPDT_OMRON-G5LE-1" H 6200 2700 50  0001 L CNN
+F 3 "" H 6200 2400 50  0001 L CNN
+	1    5550 2550
+	0    1    -1   0
+$EndComp
+Wire Wire Line
+	2900 2150 4000 2150
+Wire Wire Line
+	4600 2050 5450 2050
+Wire Wire Line
+	5450 2050 5450 2150
+Wire Wire Line
+	4750 2900 4750 3250
+Wire Wire Line
+	4750 3250 4600 3250
+Wire Wire Line
+	4600 2250 4850 2250
+Wire Wire Line
+	4850 2250 4850 1300
+Wire Wire Line
+	4850 1300 5050 1300
+Text HLabel 5050 1300 2    60   Output ~ 0
+IMD_FLT_12V_LED_H
+$Comp
+L LED D?
+U 1 1 5A09EA5C
+P 4100 4550
+F 0 "D?" H 4100 4650 50  0000 C CNN
+F 1 "LED" H 4100 4450 50  0000 C CNN
+F 2 "" H 4100 4550 50  0001 C CNN
+F 3 "" H 4100 4550 50  0001 C CNN
+	1    4100 4550
+	-1   0    0    1
+$EndComp
+$Comp
+L R R?
+U 1 1 5A09EADD
+P 4550 4550
+F 0 "R?" V 4630 4550 50  0000 C CNN
+F 1 "R" V 4550 4550 50  0000 C CNN
+F 2 "" V 4480 4550 50  0001 C CNN
+F 3 "" H 4550 4550 50  0001 C CNN
+	1    4550 4550
+	0    1    1    0
+$EndComp
+Wire Wire Line
+	4250 4550 4400 4550
+Wire Wire Line
+	4700 4550 4850 4550
+Connection ~ 4850 4550
+Wire Wire Line
+	3850 4550 3950 4550
+Connection ~ 3850 4250
+$Comp
+L LED D?
+U 1 1 5A09ECFB
+P 5600 3300
+F 0 "D?" H 5600 3400 50  0000 C CNN
+F 1 "LED" H 5600 3200 50  0000 C CNN
+F 2 "" H 5600 3300 50  0001 C CNN
+F 3 "" H 5600 3300 50  0001 C CNN
+	1    5600 3300
+	-1   0    0    1
+$EndComp
+$Comp
+L R R?
+U 1 1 5A09ED01
+P 6050 3300
+F 0 "R?" V 6130 3300 50  0000 C CNN
+F 1 "R" V 6050 3300 50  0000 C CNN
+F 2 "" V 5980 3300 50  0001 C CNN
+F 3 "" H 6050 3300 50  0001 C CNN
+	1    6050 3300
+	0    1    1    0
+$EndComp
+Wire Wire Line
+	5750 3300 5900 3300
+Wire Wire Line
+	6350 3300 6200 3300
+Wire Wire Line
+	5350 3300 5450 3300
+Wire Wire Line
+	5350 2550 5350 3300
+Connection ~ 5350 2550
+Connection ~ 5350 2950
+Wire Wire Line
+	6350 2550 6350 3300
+Connection ~ 6350 2550
+Connection ~ 6350 2950
 $EndSCHEMATC
