File: ShutdownCircuit.sch (KiCad schematic (older format))
At the start: 12 parts, among them K1 IMD_RELAY, K2 IMD_LATCH, K3 BMS_RELAY, Q3 Q_NMOS_DGS, Q4 Q_NMOS_DGS

Commit message: beginning board design
Parts:
- D1: value LED -> IMD_OK; footprint (none) -> LEDs:LED_0805_HandSoldering
- D2, D4: footprint (none) -> Diodes_SMD:D_SOT-23_ANK
- D3: value LED -> BMS_OK; footprint (none) -> LEDs:LED_0805_HandSoldering
- F13: renamed from F12; footprint (none) -> Fuse_Holders_and_Fuses:BladeFuse-Mini_Keystone_3568
- renumbered R5 to R10, R4 to R9
Changed lines of the file:
@@
 $EndDescr
 $Comp
-L +12V #PWR17
+L +12V #PWR038
 U 1 1 5A022276
 P 2900 2150
-F 0 "#PWR17" H 2900 2000 50  0001 C CNN
+F 0 "#PWR038" H 2900 2000 50  0001 C CNN
 F 1 "+12V" H 2900 2290 50  0000 C CNN
 F 2 "" H 2900 2150 50  0001 C CNN
@@
 $EndComp
 $Comp
-L +12V #PWR18
+L +12V #PWR039
 U 1 1 5A02229A
 P 3050 3350
-F 0 "#PWR18" H 3050 3200 50  0001 C CNN
+F 0 "#PWR039" H 3050 3200 50  0001 C CNN
 F 1 "+12V" H 3050 3490 50  0000 C CNN
 F 2 "" H 3050 3350 50  0001 C CNN
@@
 $EndComp
 $Comp
-L +12V #PWR20
+L +12V #PWR040
 U 1 1 5A0222EA
 P 5250 2550
-F 0 "#PWR20" H 5250 2400 50  0001 C CNN
+F 0 "#PWR040" H 5250 2400 50  0001 C CNN
 F 1 "+12V" H 5250 2690 50  0000 C CNN
 F 2 "" H 5250 2550 50  0001 C CNN
@@
 F 0 "D2" H 4300 4350 50  0000 C CNN
 F 1 "IMD_FLYBACK" H 4300 4150 50  0000 C CNN
-F 2 "" H 4300 4250 50  0001 C CNN
+F 2 "Diodes_SMD:D_SOT-23_ANK" H 4300 4250 50  0001 C CNN
 F 3 "" H 4300 4250 50  0001 C CNN
 	1    4300 4250
@@
 $EndComp
 $Comp
-L GND #PWR19
+L GND #PWR041
 U 1 1 5A022431
 P 4850 5250
-F 0 "#PWR19" H 4850 5000 50  0001 C CNN
+F 0 "#PWR041" H 4850 5000 50  0001 C CNN
 F 1 "GND" H 4850 5100 50  0000 C CNN
 F 2 "" H 4850 5250 50  0001 C CNN
@@
 F 0 "D4" H 5750 3050 50  0000 C CNN
 F 1 "BMS_FLYBACK" H 5750 2850 50  0000 C CNN
-F 2 "" H 5750 2950 50  0001 C CNN
+F 2 "Diodes_SMD:D_SOT-23_ANK" H 5750 2950 50  0001 C CNN
 F 3 "" H 5750 2950 50  0001 C CNN
 	1    5750 2950
@@
 P 4100 4550
 F 0 "D1" H 4100 4650 50  0000 C CNN
-F 1 "LED" H 4100 4450 50  0000 C CNN
-F 2 "" H 4100 4550 50  0001 C CNN
+F 1 "IMD_OK" H 4100 4450 50  0000 C CNN
+F 2 "LEDs:LED_0805_HandSoldering" H 4100 4550 50  0001 C CNN
 F 3 "" H 4100 4550 50  0001 C CNN
 	1    4100 4550
@@
 $EndComp
 $Comp
-L R R4
+L R R9
 U 1 1 5A09EADD
 P 4550 4550
-F 0 "R4" V 4630 4550 50  0000 C CNN
+F 0 "R9" V 4630 4550 50  0000 C CNN
 F 1 "R" V 4550 4550 50  0000 C CNN
 F 2 "" V 4480 4550 50  0001 C CNN
@@
 P 5600 3300
 F 0 "D3" H 5600 3400 50  0000 C CNN
-F 1 "LED" H 5600 3200 50  0000 C CNN
-F 2 "" H 5600 3300 50  0001 C CNN
+F 1 "BMS_OK" H 5600 3200 50  0000 C CNN
+F 2 "LEDs:LED_0805_HandSoldering" H 5600 3300 50  0001 C CNN
 F 3 "" H 5600 3300 50  0001 C CNN
 	1    5600 3300
@@
 $EndComp
 $Comp
-L R R5
+L R R10
 U 1 1 5A09ED01
 P 6050 3300
-F 0 "R5" V 6130 3300 50  0000 C CNN
+F 0 "R10" V 6130 3300 50  0000 C CNN
 F 1 "R" V 6050 3300 50  0000 C CNN
 F 2 "" V 5980 3300 50  0001 C CNN
@@
 Connection ~ 6350 2950
 $Comp
-L Fuse F12
+L Fuse F13
 U 1 1 5A122E62
 P 3500 2150
-F 0 "F12" V 3580 2150 50  0000 C CNN
+F 0 "F13" V 3580 2150 50  0000 C CNN
 F 1 "SD_FUSE" V 3425 2150 50  0000 C CNN
-F 2 "" V 3430 2150 50  0001 C CNN
+F 2 "Fuse_Holders_and_Fuses:BladeFuse-Mini_Keystone_3568" V 3430 2150 50  0001 C CNN
 F 3 "" H 3500 2150 50  0001 C CNN
 	1    3500 2150

Commit message: stuff
Other:
- note added: "5A"
Changed lines of the file:
@@
 $Descr A4 11693 8268
 encoding utf-8
-Sheet 2 4
+Sheet 4 4
 Title ""
 Date ""
@@
 Text HLabel 3250 3000 0    60   Input ~ 0
 IMD_RST+
+Text Notes 3450 2050 0    60   ~ 0
+5A
 $EndSCHEMATC

Commit message: winter break changes
Parts:
- D1, D3: footprint LEDs:LED_0805_HandSoldering -> LEDs:LED_0603_HandSoldering
- Q3, Q4: footprint (none) -> TO_SOT_Packages_SMD:TO-263-2
- R10, R9: footprint (none) -> Resistors_SMD:R_0603_HandSoldering
Changed lines of the file:
@@
 F 0 "Q3" H 4950 4900 50  0000 L CNN
 F 1 "Q_NMOS_DGS" H 4950 4800 50  0000 L CNN
-F 2 "" H 4950 4950 50  0001 C CNN
+F 2 "TO_SOT_Packages_SMD:TO-263-2" H 4950 4950 50  0001 C CNN
 F 3 "" H 4750 4850 50  0001 C CNN
 	1    4750 4850
@@
 F 0 "Q4" H 6600 4900 50  0000 L CNN
 F 1 "Q_NMOS_DGS" H 6600 4800 50  0000 L CNN
-F 2 "" H 6600 4950 50  0001 C CNN
+F 2 "TO_SOT_Packages_SMD:TO-263-2" H 6600 4950 50  0001 C CNN
 F 3 "" H 6400 4850 50  0001 C CNN
 	1    6400 4850
@@
 F 0 "D1" H 4100 4650 50  0000 C CNN
 F 1 "IMD_OK" H 4100 4450 50  0000 C CNN
-F 2 "LEDs:LED_0805_HandSoldering" H 4100 4550 50  0001 C CNN
+F 2 "LEDs:LED_0603_HandSoldering" H 4100 4550 50  0001 C CNN
 F 3 "" H 4100 4550 50  0001 C CNN
 	1    4100 4550
@@
 F 0 "R9" V 4630 4550 50  0000 C CNN
 F 1 "R" V 4550 4550 50  0000 C CNN
-F 2 "" V 4480 4550 50  0001 C CNN
+F 2 "Resistors_SMD:R_0603_HandSoldering" V 4480 4550 50  0001 C CNN
 F 3 "" H 4550 4550 50  0001 C CNN
 	1    4550 4550
@@
 F 0 "D3" H 5600 3400 50  0000 C CNN
 F 1 "BMS_OK" H 5600 3200 50  0000 C CNN
-F 2 "LEDs:LED_0805_HandSoldering" H 5600 3300 50  0001 C CNN
+F 2 "LEDs:LED_0603_HandSoldering" H 5600 3300 50  0001 C CNN
 F 3 "" H 5600 3300 50  0001 C CNN
 	1    5600 3300
@@
 F 0 "R10" V 6130 3300 50  0000 C CNN
 F 1 "R" V 6050 3300 50  0000 C CNN
-F 2 "" V 5980 3300 50  0001 C CNN
+F 2 "Resistors_SMD:R_0603_HandSoldering" V 5980 3300 50  0001 C CNN
 F 3 "" H 6050 3300 50  0001 C CNN
 	1    6050 3300

Commit message: finished routing
Parts:
- removed Q3, Q4: Q_NMOS_DGS, TO_SOT_Packages_SMD:TO-263-2, symbol Q_NMOS_DGS
- added Q3, Q4: Q_NMOS_GDS, TO_SOT_Packages_SMD:TO-252-2, symbol Q_NMOS_GDS
- added R11, R3: 10k, Resistors_SMD:R_0805_HandSoldering, symbol R
- D1, D3: footprint LEDs:LED_0603_HandSoldering -> LEDs:LED_0805_HandSoldering
- R10, R9: footprint Resistors_SMD:R_0603_HandSoldering -> Resistors_SMD:R_0805_HandSoldering
Connections:
- wire segments 38 -> 42
Changed lines of the file:
@@
 $EndDescr
 $Comp
-L +12V #PWR042
+L +12V #PWR050
 U 1 1 5A022276
 P 2900 2150
-F 0 "#PWR042" H 2900 2000 50  0001 C CNN
+F 0 "#PWR050" H 2900 2000 50  0001 C CNN
 F 1 "+12V" H 2900 2290 50  0000 C CNN
 F 2 "" H 2900 2150 50  0001 C CNN
@@
 $EndComp
 $Comp
-L +12V #PWR043
+L +12V #PWR051
 U 1 1 5A02229A
 P 3050 3350
-F 0 "#PWR043" H 3050 3200 50  0001 C CNN
+F 0 "#PWR051" H 3050 3200 50  0001 C CNN
 F 1 "+12V" H 3050 3490 50  0000 C CNN
 F 2 "" H 3050 3350 50  0001 C CNN
@@
 $EndComp
 $Comp
-L +12V #PWR044
+L +12V #PWR052
 U 1 1 5A0222EA
 P 5250 2550
-F 0 "#PWR044" H 5250 2400 50  0001 C CNN
+F 0 "#PWR052" H 5250 2400 50  0001 C CNN
 F 1 "+12V" H 5250 2690 50  0000 C CNN
 F 2 "" H 5250 2550 50  0001 C CNN
@@
 $EndComp
 $Comp
-L GND #PWR045
+L GND #PWR053
 U 1 1 5A022431
 P 4850 5250
-F 0 "#PWR045" H 4850 5000 50  0001 C CNN
+F 0 "#PWR053" H 4850 5000 50  0001 C CNN
 F 1 "GND" H 4850 5100 50  0000 C CNN
 F 2 "" H 4850 5250 50  0001 C CNN
@@
 	1    0    0    -1
 $EndComp
-$Comp
-L Q_NMOS_DGS Q3
-U 1 1 5A022451
-P 4750 4850
-F 0 "Q3" H 4950 4900 50  0000 L CNN
-F 1 "Q_NMOS_DGS" H 4950 4800 50  0000 L CNN
-F 2 "TO_SOT_Packages_SMD:TO-263-2" H 4950 4950 50  0001 C CNN
-F 3 "" H 4750 4850 50  0001 C CNN
-	1    4750 4850
-	1    0    0    -1
-$EndComp
-$Comp
-L Q_NMOS_DGS Q4
-U 1 1 5A0225B4
-P 6400 4850
-F 0 "Q4" H 6600 4900 50  0000 L CNN
-F 1 "Q_NMOS_DGS" H 6600 4800 50  0000 L CNN
-F 2 "TO_SOT_Packages_SMD:TO-263-2" H 6600 4950 50  0001 C CNN
-F 3 "" H 6400 4850 50  0001 C CNN
-	1    6400 4850
-	1    0    0    -1
-$EndComp
-Text HLabel 4550 4850 0    60   Input ~ 0
+Text HLabel 4350 4850 0    60   Input ~ 0
 IMD_FLT_5V_L
-Text HLabel 6200 4850 0    60   Input ~ 0
+Text HLabel 6050 4850 0    60   Input ~ 0
 BMS_FLT_5V_L
 Text HLabel 6050 2050 2    60   Output ~ 0
@@
 Connection ~ 3850 3000
 Wire Wire Line
-	6500 5050 6500 5200
-Wire Wire Line
-	6500 5200 4850 5200
+	6500 5200 6500 5050
+Wire Wire Line
+	4450 5200 6500 5200
 Connection ~ 4850 5200
 Wire Wire Line
@@
 F 0 "D1" H 4100 4650 50  0000 C CNN
 F 1 "IMD_OK" H 4100 4450 50  0000 C CNN
-F 2 "LEDs:LED_0603_HandSoldering" H 4100 4550 50  0001 C CNN
+F 2 "LEDs:LED_0805_HandSoldering" H 4100 4550 50  0001 C CNN
 F 3 "" H 4100 4550 50  0001 C CNN
 	1    4100 4550
@@
 F 0 "R9" V 4630 4550 50  0000 C CNN
 F 1 "R" V 4550 4550 50  0000 C CNN
-F 2 "Resistors_SMD:R_0603_HandSoldering" V 4480 4550 50  0001 C CNN
+F 2 "Resistors_SMD:R_0805_HandSoldering" V 4480 4550 50  0001 C CNN
 F 3 "" H 4550 4550 50  0001 C CNN
 	1    4550 4550
@@
 F 0 "D3" H 5600 3400 50  0000 C CNN
 F 1 "BMS_OK" H 5600 3200 50  0000 C CNN
-F 2 "LEDs:LED_0603_HandSoldering" H 5600 3300 50  0001 C CNN
+F 2 "LEDs:LED_0805_HandSoldering" H 5600 3300 50  0001 C CNN
 F 3 "" H 5600 3300 50  0001 C CNN
 	1    5600 3300
@@
 F 0 "R10" V 6130 3300 50  0000 C CNN
 F 1 "R" V 6050 3300 50  0000 C CNN
-F 2 "Resistors_SMD:R_0603_HandSoldering" V 5980 3300 50  0001 C CNN
+F 2 "Resistors_SMD:R_0805_HandSoldering" V 5980 3300 50  0001 C CNN
 F 3 "" H 6050 3300 50  0001 C CNN
 	1    6050 3300
@@
 Text Notes 3450 2050 0    60   ~ 0
 5A
+$Comp
+L Q_NMOS_GDS Q4
+U 1 1 5A66D7B9
+P 6400 4850
+F 0 "Q4" H 6600 4900 50  0000 L CNN
+F 1 "Q_NMOS_GDS" H 6600 4800 50  0000 L CNN
+F 2 "TO_SOT_Packages_SMD:TO-252-2" H 6600 4950 50  0001 C CNN
+F 3 "" H 6400 4850 50  0001 C CNN
+	1    6400 4850
+	1    0    0    -1
+$EndComp
+$Comp
+L Q_NMOS_GDS Q3
+U 1 1 5A66D81E
+P 4750 4850
+F 0 "Q3" H 4950 4900 50  0000 L CNN
+F 1 "Q_NMOS_GDS" H 4950 4800 50  0000 L CNN
+F 2 "TO_SOT_Packages_SMD:TO-252-2" H 4950 4950 50  0001 C CNN
+F 3 "" H 4750 4850 50  0001 C CNN
+	1    4750 4850
+	1    0    0    -1
+$EndComp
+$Comp
+L R R11
+U 1 1 5A677D71
+P 6100 5050
+F 0 "R11" V 6180 5050 50  0000 C CNN
+F 1 "10k" V 6100 5050 50  0000 C CNN
+F 2 "Resistors_SMD:R_0805_HandSoldering" V 6030 5050 50  0001 C CNN
+F 3 "" H 6100 5050 50  0001 C CNN
+	1    6100 5050
+	1    0    0    -1
+$EndComp
+Connection ~ 6100 5200
+Wire Wire Line
+	6050 4850 6200 4850
+Wire Wire Line
+	6100 4900 6100 4850
+Connection ~ 6100 4850
+$Comp
+L R R3
+U 1 1 5A678B3E
+P 4450 5050
+F 0 "R3" V 4530 5050 50  0000 C CNN
+F 1 "10k" V 4450 5050 50  0000 C CNN
+F 2 "Resistors_SMD:R_0805_HandSoldering" V 4380 5050 50  0001 C CNN
+F 3 "" H 4450 5050 50  0001 C CNN
+	1    4450 5050
+	1    0    0    -1
+$EndComp
+Wire Wire Line
+	4350 4850 4550 4850
+Wire Wire Line
+	4450 4900 4450 4850
+Connection ~ 4450 4850
 $EndSCHEMATC

Commit message: final design competition 2018
Parts:
- R10, R9: value R -> 100k
Changed lines of the file:
@@
 P 4550 4550
 F 0 "R9" V 4630 4550 50  0000 C CNN
-F 1 "R" V 4550 4550 50  0000 C CNN
+F 1 "100k" V 4550 4550 50  0000 C CNN
 F 2 "Resistors_SMD:R_0805_HandSoldering" V 4480 4550 50  0001 C CNN
 F 3 "" H 4550 4550 50  0001 C CNN
@@
 P 6050 3300
 F 0 "R10" V 6130 3300 50  0000 C CNN
-F 1 "R" V 6050 3300 50  0000 C CNN
+F 1 "100k" V 6050 3300 50  0000 C CNN
 F 2 "Resistors_SMD:R_0805_HandSoldering" V 5980 3300 50  0001 C CNN
 F 3 "" H 6050 3300 50  0001 C CNN
