File: Motherboard.sch (KiCad schematic (older format))
At the start: 18 parts, among them Q1 Q_NMOS_DGS, Q2 Q_NMOS_DGS, U1 LM7805_TO220

Commit message: added noel's revisions
Parts:
- added J?: Conn_01x35_Male, symbol Conn_01x35_Male
- gave numbers to parts that had none: 2
- renumbered F7 to F10, F9 to F11, F10 to F3, F2 to F4, F3 to F5, F4 to F6, F5 to F7, F6 to F8, F8 to F9, R3 to R2, R2 to R3
Connections:
- net labels removed: SEVCON_BRK, SEVCON_THR
- wire segments 64 -> 59
Other:
- moved on the sheet: F10, F11, F12, F3, F5, F6, F7, F8, F9

Commit message: added charger sd logic
Parts:
- removed J?: Conn_01x35_Male, symbol Conn_01x35_Male
- added J? (x3): Conn_01x14_Male, symbol Conn_01x14_Male
- added U?: 74HC00, symbol 74HC00
Connections:
- net labels added: CHARGER_SD
- wire segments 59 -> 63
Other:
- note added: "GLV"
- note added: "Peripheral"
- note added: "TS/SD"
- moved on the sheet: F10, F11, F12, F3, F5, F6, F7, F8, F9
