File: Motherboard.sch (KiCad schematic (older format))
At the start: 24 parts, among them J1 Conn_01x16_Male, J2 Conn_01x04_Male, J3 Conn_01x14_Male, J4 Conn_01x14_Male, J5 Conn_01x14_Male, Q1 Q_NMOS_DGS, Q2 Q_NMOS_DGS, U1 LM7805_TO220, U2 74HC00

Commit message: beginning board design
Parts:
- F1, F2: footprint (none) -> Fuse_Holders_and_Fuses:BladeFuse-Mini_Keystone_3568
- F10: renamed from F?; footprint (none) -> Fuse_Holders_and_Fuses:BladeFuse-Mini_Keystone_3568
- F11: renamed from F4; footprint (none) -> Fuse_Holders_and_Fuses:BladeFuse-Mini_Keystone_3568
- F12: renamed from F5; footprint (none) -> Fuse_Holders_and_Fuses:BladeFuse-Mini_Keystone_3568
- F3: renamed from F6; footprint (none) -> Fuse_Holders_and_Fuses:BladeFuse-Mini_Keystone_3568
- F4: renamed from F7; footprint (none) -> Fuse_Holders_and_Fuses:BladeFuse-Mini_Keystone_3568
- F5: renamed from F8; footprint (none) -> Fuse_Holders_and_Fuses:BladeFuse-Mini_Keystone_3568
- F6: renamed from F9; footprint (none) -> Fuse_Holders_and_Fuses:BladeFuse-Mini_Keystone_3568
- F7: renamed from F10; footprint (none) -> Fuse_Holders_and_Fuses:BladeFuse-Mini_Keystone_3568
- F8: renamed from F11; footprint (none) -> Fuse_Holders_and_Fuses:BladeFuse-Mini_Keystone_3568
- F9: renamed from F3; footprint (none) -> Fuse_Holders_and_Fuses:BladeFuse-Mini_Keystone_3568
- J3, J4, J5: footprint (none) -> TuftsRacing2018:AMP14
- R1, R2, R3: footprint (none) -> Resistors_SMD:R_0805_HandSoldering
- U1: footprint TO_SOT_Packages_THT:TO-220_Vertical -> Power_Integrations:TO-220
- U2: footprint (none) -> Housings_DIP:DIP-14_W8.89mm_SMDSocket_LongPads

Commit message: working on bms connectors
Parts:
- removed R3: 10k, Resistors_SMD:R_0805_HandSoldering, symbol R
- added J?: Conn_01x05_Male, symbol Conn_01x05_Male
Connections:
- wire segments 62 -> 59
- no-connect marks 0 -> 4
Other:
- note added: "+12V charging"
- note added: "+12V discharging"
- note added: "src?"
- note removed: "BMS"
- moved on the sheet: F2
Changed lines of the file:
@@
 L Fuse F2
 U 1 1 5A030C01
-P 6750 1000
-F 0 "F2" V 6830 1000 50  0000 C CNN
-F 1 "BMS_FUSE" V 6675 1000 50  0000 C CNN
-F 2 "Fuse_Holders_and_Fuses:BladeFuse-Mini_Keystone_3568" V 6680 1000 50  0001 C CNN
-F 3 "" H 6750 1000 50  0001 C CNN
-	1    6750 1000
+P 6400 1250
+F 0 "F2" V 6480 1250 50  0000 C CNN
+F 1 "BMS_FUSE" V 6325 1250 50  0000 C CNN
+F 2 "Fuse_Holders_and_Fuses:BladeFuse-Mini_Keystone_3568" V 6330 1250 50  0001 C CNN
+F 3 "" H 6400 1250 50  0001 C CNN
+	1    6400 1250
 	0    1    1    0
 $EndComp
@@
 Text Label 9850 3550 2    60   ~ 0
 IMD_FLT
-Text Label 7500 1400 2    60   ~ 0
+Text Label 8150 2100 2    60   ~ 0
 BMS_FLT
 Text Label 9850 5550 2    60   ~ 0
@@
 Text Label 9850 4750 2    60   ~ 0
 FAN-
-Text Label 7500 1100 2    60   ~ 0
+Text Label 8150 1400 2    60   ~ 0
 CONTACT_REQ
-Text Label 7500 1200 2    60   ~ 0
+Text Label 6400 2550 2    60   ~ 0
 FAN_PWM
-Text Label 7500 1300 2    60   ~ 0
+Text Label 8150 2200 2    60   ~ 0
 SOC
 Text Label 7950 3050 2    60   ~ 0
@@
 Text Notes 10700 4750 2    60   ~ 0
 battery_fans
-Text Notes 7800 1250 2    60   ~ 0
-BMS
-$Comp
-L GND #PWR09
-U 1 1 5A0580F9
-P 7350 1850
-F 0 "#PWR09" H 7350 1600 50  0001 C CNN
-F 1 "GND" H 7350 1700 50  0000 C CNN
-F 2 "" H 7350 1850 50  0001 C CNN
-F 3 "" H 7350 1850 50  0001 C CNN
-	1    7350 1850
-	1    0    0    -1
-$EndComp
 Text Label 9850 2650 2    60   ~ 0
 K1
@@
 batt_relays-
 $Comp
-L R R3
-U 1 1 5A059781
-P 6450 1200
-F 0 "R3" V 6530 1200 50  0000 C CNN
-F 1 "10k" V 6450 1200 50  0000 C CNN
-F 2 "Resistors_SMD:R_0805_HandSoldering" V 6380 1200 50  0001 C CNN
-F 3 "" H 6450 1200 50  0001 C CNN
-	1    6450 1200
-	1    0    0    -1
-$EndComp
-$Comp
 L +12V #PWR010
 U 1 1 5A059A94
-P 6350 1000
-F 0 "#PWR010" H 6350 850 50  0001 C CNN
-F 1 "+12V" H 6350 1140 50  0000 C CNN
-F 2 "" H 6350 1000 50  0001 C CNN
-F 3 "" H 6350 1000 50  0001 C CNN
-	1    6350 1000
+P 6000 1250
+F 0 "#PWR010" H 6000 1100 50  0001 C CNN
+F 1 "+12V" H 6000 1390 50  0000 C CNN
+F 2 "" H 6000 1250 50  0001 C CNN
+F 3 "" H 6000 1250 50  0001 C CNN
+	1    6000 1250
 	1    0    0    -1
 $EndComp
@@
 	9150 3450 8900 3450
 Wire Wire Line
-	6900 1000 7500 1000
+	6550 1250 7150 1250
 Wire Wire Line
 	9450 3450 9850 3450
@@
 	8950 1350 9850 1350
 Wire Wire Line
-	7500 1800 7350 1800
-Wire Wire Line
-	7350 1800 7350 1850
-Wire Wire Line
-	6450 1400 7500 1400
-Wire Wire Line
-	6450 1400 6450 1350
-Wire Wire Line
 	9850 1750 9850 1750
 Wire Wire Line
-	6350 1000 6600 1000
-Wire Wire Line
-	6450 1000 6450 1050
-Connection ~ 6450 1000
+	6000 1250 6250 1250
 Wire Wire Line
 	6250 4300 6400 4300
@@
 L Conn_01x16_Male J1
 U 1 1 5A18A953
-P 7950 1700
-F 0 "J1" H 7950 2500 50  0000 C CNN
-F 1 "Conn_01x16_Male" H 7950 800 50  0000 C CNN
-F 2 "" H 7950 1700 50  0001 C CNN
-F 3 "" H 7950 1700 50  0001 C CNN
-	1    7950 1700
-	1    0    0    -1
+P 8350 1700
+F 0 "J1" H 8350 2500 50  0000 C CNN
+F 1 "Conn_01x16_Male" H 8350 800 50  0000 C CNN
+F 2 "" H 8350 1700 50  0001 C CNN
+F 3 "" H 8350 1700 50  0001 C CNN
+	1    8350 1700
+	-1   0    0    -1
 $EndComp
 $Comp
@@
 Wire Wire Line
 	9450 950  9850 950
+$Comp
+L GND #PWR?
+U 1 1 5A1EF9E0
+P 8150 1000
+F 0 "#PWR?" H 8150 750 50  0001 C CNN
+F 1 "GND" H 8150 850 50  0000 C CNN
+F 2 "" H 8150 1000 50  0001 C CNN
+F 3 "" H 8150 1000 50  0001 C CNN
+	1    8150 1000
+	0    1    1    0
+$EndComp
+$Comp
+L GND #PWR?
+U 1 1 5A1EFAC0
+P 8150 1800
+F 0 "#PWR?" H 8150 1550 50  0001 C CNN
+F 1 "GND" H 8150 1650 50  0000 C CNN
+F 2 "" H 8150 1800 50  0001 C CNN
+F 3 "" H 8150 1800 50  0001 C CNN
+	1    8150 1800
+	0    1    1    0
+$EndComp
+Wire Wire Line
+	8150 1200 7700 1200
+Wire Wire Line
+	8150 1300 7700 1300
+Text Notes 7150 1200 0    60   ~ 0
++12V discharging
+Text Notes 7200 1300 0    60   ~ 0
++12V charging
+Text Notes 7600 1500 0    60   ~ 0
+src?
+$Comp
+L Conn_01x05_Male J?
+U 1 1 5A1F5EC6
+P 6600 2450
+F 0 "J?" H 6600 2750 50  0000 C CNN
+F 1 "Conn_01x05_Male" H 6600 2150 50  0000 C CNN
+F 2 "" H 6600 2450 50  0001 C CNN
+F 3 "" H 6600 2450 50  0001 C CNN
+	1    6600 2450
+	-1   0    0    -1
+$EndComp
+$Comp
+L GND #PWR?
+U 1 1 5A1F6F20
+P 6400 2250
+F 0 "#PWR?" H 6400 2000 50  0001 C CNN
+F 1 "GND" H 6400 2100 50  0000 C CNN
+F 2 "" H 6400 2250 50  0001 C CNN
+F 3 "" H 6400 2250 50  0001 C CNN
+	1    6400 2250
+	0    1    1    0
+$EndComp
+NoConn ~ 6400 2350
+NoConn ~ 6400 2450
+NoConn ~ 6400 2650
+NoConn ~ 7950 2950
 $EndSCHEMATC

Commit message: stuff
Parts:
- gave numbers to parts that had none: 1
Other:
- note added: "15A"
- note added: "2A"
- note added: "4A"
- note added: "5A"
- note added: "7.5A"
- note added: "check pn"
- note added: "sd_ckt"
Changed lines of the file:
@@
 SD_CKT+
 $Comp
-L GND #PWR01
+L GND #PWR2
 U 1 1 5A02DEC9
 P 3250 3400
-F 0 "#PWR01" H 3250 3150 50  0001 C CNN
+F 0 "#PWR2" H 3250 3150 50  0001 C CNN
 F 1 "GND" H 3250 3250 50  0000 C CNN
 F 2 "" H 3250 3400 50  0001 C CNN
@@
 $EndComp
 $Comp
-L +5V #PWR02
+L +5V #PWR3
 U 1 1 5A02DFBF
 P 4000 2900
-F 0 "#PWR02" H 4000 2750 50  0001 C CNN
+F 0 "#PWR3" H 4000 2750 50  0001 C CNN
 F 1 "+5V" H 4000 3040 50  0000 C CNN
 F 2 "" H 4000 2900 50  0001 C CNN
@@
 $EndComp
 $Comp
-L +12V #PWR03
+L +12V #PWR1
 U 1 1 5A02E07D
 P 2900 2900
-F 0 "#PWR03" H 2900 2750 50  0001 C CNN
+F 0 "#PWR1" H 2900 2750 50  0001 C CNN
 F 1 "+12V" H 2900 3040 50  0000 C CNN
 F 2 "" H 2900 2900 50  0001 C CNN
@@
 $EndComp
 $Comp
-L GND #PWR04
+L GND #PWR4
 U 1 1 5A02F04B
 P 5100 4650
-F 0 "#PWR04" H 5100 4400 50  0001 C CNN
+F 0 "#PWR4" H 5100 4400 50  0001 C CNN
 F 1 "GND" H 5100 4500 50  0000 C CNN
 F 2 "" H 5100 4650 50  0001 C CNN
@@
 IMD_FLT_12V_LED_H
 $Comp
-L +5V #PWR05
+L +5V #PWR14
 U 1 1 5A046BA9
 P 8900 2050
-F 0 "#PWR05" H 8900 1900 50  0001 C CNN
+F 0 "#PWR14" H 8900 1900 50  0001 C CNN
 F 1 "+5V" H 8900 2190 50  0000 C CNN
 F 2 "" H 8900 2050 50  0001 C CNN
@@
 $EndComp
 $Comp
-L GND #PWR06
+L GND #PWR16
 U 1 1 5A046C61
 P 8950 1350
-F 0 "#PWR06" H 8950 1100 50  0001 C CNN
+F 0 "#PWR16" H 8950 1100 50  0001 C CNN
 F 1 "GND" H 8950 1200 50  0000 C CNN
 F 2 "" H 8950 1350 50  0001 C CNN
@@
 	0    1    1    0
 $EndComp
-Text Notes 10750 1200 2    60   ~ 0
+Text Notes 10750 1300 2    60   ~ 0
 steering wheel
 Text Notes 10250 3200 0    60   ~ 0
@@
 SEVCON_FLT
 $Comp
-L GND #PWR07
+L GND #PWR20
 U 1 1 5A048248
 P 9850 3350
-F 0 "#PWR07" H 9850 3100 50  0001 C CNN
+F 0 "#PWR20" H 9850 3100 50  0001 C CNN
 F 1 "GND" H 9850 3200 50  0000 C CNN
 F 2 "" H 9850 3350 50  0001 C CNN
@@
 $EndComp
 $Comp
-L GND #PWR08
+L GND #PWR17
 U 1 1 5A04A097
 P 9400 3650
-F 0 "#PWR08" H 9400 3400 50  0001 C CNN
+F 0 "#PWR17" H 9400 3400 50  0001 C CNN
 F 1 "GND" H 9400 3500 50  0000 C CNN
 F 2 "" H 9400 3650 50  0001 C CNN
@@
 batt_relays-
 $Comp
-L +12V #PWR010
+L +12V #PWR5
 U 1 1 5A059A94
 P 6000 1250
-F 0 "#PWR010" H 6000 1100 50  0001 C CNN
+F 0 "#PWR5" H 6000 1100 50  0001 C CNN
 F 1 "+12V" H 6000 1390 50  0000 C CNN
 F 2 "" H 6000 1250 50  0001 C CNN
@@
 SCL
 $Comp
-L GND #PWR011
+L GND #PWR19
 U 1 1 5A05EFDD
 P 9850 1950
-F 0 "#PWR011" H 9850 1700 50  0001 C CNN
+F 0 "#PWR19" H 9850 1700 50  0001 C CNN
 F 1 "GND" H 9850 1800 50  0000 C CNN
 F 2 "" H 9850 1950 50  0001 C CNN
@@
 	0    1    1    0
 $EndComp
-Text Notes 10500 1650 2    60   ~ 0
+Text Notes 10500 1850 2    60   ~ 0
 daq
 $Comp
@@
 $EndComp
 $Comp
-L GND #PWR012
+L GND #PWR7
 U 1 1 5A061CAC
 P 6700 4650
-F 0 "#PWR012" H 6700 4400 50  0001 C CNN
+F 0 "#PWR7" H 6700 4400 50  0001 C CNN
 F 1 "GND" H 6700 4500 50  0000 C CNN
 F 2 "" H 6700 4650 50  0001 C CNN
@@
 $EndComp
 $Comp
-L +12V #PWR013
+L +12V #PWR11
 U 1 1 5A066D1D
 P 8700 2950
-F 0 "#PWR013" H 8700 2800 50  0001 C CNN
+F 0 "#PWR11" H 8700 2800 50  0001 C CNN
 F 1 "+12V" H 8700 3090 50  0000 C CNN
 F 2 "" H 8700 2950 50  0001 C CNN
@@
 $EndComp
 $Comp
-L +12V #PWR014
+L +12V #PWR15
 U 1 1 5A066DDB
 P 8900 3450
-F 0 "#PWR014" H 8900 3300 50  0001 C CNN
+F 0 "#PWR15" H 8900 3300 50  0001 C CNN
 F 1 "+12V" H 8900 3590 50  0000 C CNN
 F 2 "" H 8900 3450 50  0001 C CNN
@@
 Text Notes 10600 4950 2    60   ~ 0
 brk_light
-Text Notes 10600 2000 2    60   ~ 0
+Text Notes 10650 2200 2    60   ~ 0
 pedal_box
 $Comp
@@
 Connection ~ 8600 4650
 $Comp
-L +12V #PWR015
+L +12V #PWR13
 U 1 1 5A17D849
 P 8900 1650
-F 0 "#PWR015" H 8900 1500 50  0001 C CNN
+F 0 "#PWR13" H 8900 1500 50  0001 C CNN
 F 1 "+12V" H 8900 1790 50  0000 C CNN
 F 2 "" H 8900 1650 50  0001 C CNN
@@
 $EndComp
 Wire Notes Line
-	10050 900  10050 2100
-Wire Notes Line
-	10050 1400 10800 1400
-Wire Notes Line
-	10800 900  10800 2100
+	10050 900  10050 2300
+Wire Notes Line
+	10800 900  10800 2300
 Wire Notes Line
 	10800 900  10050 900
-Wire Notes Line
-	10800 1800 10050 1800
-Wire Notes Line
-	10800 2100 10050 2100
 Wire Notes Line
 	10050 4600 10800 4600
@@
 	9250 5250 9150 5250
 Wire Notes Line
-	10050 4400 10050 5300
+	10050 4400 10050 5800
 Wire Notes Line
 	10050 5300 10800 5300
 Wire Notes Line
-	10800 5300 10800 4400
+	10800 4400 10800 5800
 Wire Notes Line
 	10800 4000 10800 2600
@@
 IMD_FLT_12V_LED_H
 $Comp
-L GND #PWR016
+L GND #PWR18
 U 1 1 5A198B33
 P 9850 1550
-F 0 "#PWR016" H 9850 1300 50  0001 C CNN
+F 0 "#PWR18" H 9850 1300 50  0001 C CNN
 F 1 "GND" H 9850 1400 50  0000 C CNN
 F 2 "" H 9850 1550 50  0001 C CNN
@@
 	8850 4450 8600 4450
 $Comp
-L +12V #PWR017
+L +12V #PWR10
 U 1 1 5A066E99
 P 8600 4350
-F 0 "#PWR017" H 8600 4200 50  0001 C CNN
+F 0 "#PWR10" H 8600 4200 50  0001 C CNN
 F 1 "+12V" H 8600 4490 50  0000 C CNN
 F 2 "" H 8600 4350 50  0001 C CNN
@@
 $EndComp
 $Comp
-L +12V #PWR018
+L +12V #PWR12
 U 1 1 5A19A158
 P 8900 950
-F 0 "#PWR018" H 8900 800 50  0001 C CNN
+F 0 "#PWR12" H 8900 800 50  0001 C CNN
 F 1 "+12V" H 8900 1090 50  0000 C CNN
 F 2 "" H 8900 950 50  0001 C CNN
@@
 	9450 950  9850 950
 $Comp
-L GND #PWR?
+L GND #PWR8
 U 1 1 5A1EF9E0
 P 8150 1000
-F 0 "#PWR?" H 8150 750 50  0001 C CNN
+F 0 "#PWR8" H 8150 750 50  0001 C CNN
 F 1 "GND" H 8150 850 50  0000 C CNN
 F 2 "" H 8150 1000 50  0001 C CNN
@@
 $EndComp
 $Comp
-L GND #PWR?
+L GND #PWR9
 U 1 1 5A1EFAC0
 P 8150 1800
-F 0 "#PWR?" H 8150 1550 50  0001 C CNN
+F 0 "#PWR9" H 8150 1550 50  0001 C CNN
 F 1 "GND" H 8150 1650 50  0000 C CNN
 F 2 "" H 8150 1800 50  0001 C CNN
@@
 src?
 $Comp
-L Conn_01x05_Male J?
+L Conn_01x05_Male J8
 U 1 1 5A1F5EC6
 P 6600 2450
-F 0 "J?" H 6600 2750 50  0000 C CNN
+F 0 "J8" H 6600 2750 50  0000 C CNN
 F 1 "Conn_01x05_Male" H 6600 2150 50  0000 C CNN
 F 2 "" H 6600 2450 50  0001 C CNN
@@
 $EndComp
 $Comp
-L GND #PWR?
+L GND #PWR6
 U 1 1 5A1F6F20
 P 6400 2250
-F 0 "#PWR?" H 6400 2000 50  0001 C CNN
+F 0 "#PWR6" H 6400 2000 50  0001 C CNN
 F 1 "GND" H 6400 2100 50  0000 C CNN
 F 2 "" H 6400 2250 50  0001 C CNN
@@
 NoConn ~ 6400 2650
 NoConn ~ 7950 2950
+Text Notes 8750 3000 0    60   ~ 0
+7.5A
+Text Notes 9350 4650 0    60   ~ 0
+15A
+Text Notes 9400 4450 0    60   ~ 0
+4A
+Text Notes 9400 4850 0    60   ~ 0
+2A
+Text Notes 9350 5050 0    60   ~ 0
+check pn
+Text Notes 9400 5150 0    60   ~ 0
+5A
+Text Notes 9400 5250 0    60   ~ 0
+5A
+Text Notes 9500 3450 0    60   ~ 0
+2A
+Text Notes 6750 1250 0    60   ~ 0
+5A
+Wire Notes Line
+	10800 5800 10050 5800
+Text Notes 10250 5550 0    60   ~ 0
+sd_ckt
+Wire Notes Line
+	10050 1600 10800 1600
+Wire Notes Line
+	10050 2000 10800 2000
+Wire Notes Line
+	10800 2300 10050 2300
 $EndSCHEMATC

Commit message: beginning floorplan
Connections:
- net labels added: BATT_FAN+, BATT_FAN-, BRK_LIGHT+, LAP_TIMER+, PUMP+, RAD_FAN+, RTDS+
- net labels removed: FAN-
- no-connect marks 4 -> 5
Other:
- moved on the sheet: F1, F12, F3, F4, F5, F6, F7, F8, F9, U1

Commit message: winter break changes
Parts:
- removed J8: Conn_01x05_Male, symbol Conn_01x05_Male
- added J8: Conn_01x06_Male, Connectors_Molex:Molex_MiniFit-JR-5556-06A_2x03x4.20mm_Straight, symbol Conn_01x06_Male
- J1: footprint (none) -> Connectors_Molex:Molex_MiniFit-JR-5556-16A_2x08x4.20mm_Straight
- J2: footprint (none) -> Connectors_Molex:Molex_MiniFit-JR-5556-04A_2x02x4.20mm_Straight
- Q1, Q2: footprint (none) -> TO_SOT_Packages_SMD:TO-263-2
- R1, R2: footprint Resistors_SMD:R_0805_HandSoldering -> Resistors_SMD:R_0603_HandSoldering
Changed lines of the file:
@@
 F 0 "Q1" H 5200 4350 50  0000 L CNN
 F 1 "Q_NMOS_DGS" H 5200 4250 50  0000 L CNN
-F 2 "" H 5200 4400 50  0001 C CNN
+F 2 "TO_SOT_Packages_SMD:TO-263-2" H 5200 4400 50  0001 C CNN
 F 3 "" H 5000 4300 50  0001 C CNN
 	1    5000 4300
@@
 Text Label 8150 1400 2    60   ~ 0
 CONTACT_REQ
-Text Label 6400 2550 2    60   ~ 0
+Text Label 6700 2450 2    60   ~ 0
 FAN_PWM
 Text Label 8150 2200 2    60   ~ 0
@@
 F 0 "Q2" H 6800 4350 50  0000 L CNN
 F 1 "Q_NMOS_DGS" H 6800 4250 50  0000 L CNN
-F 2 "" H 6800 4400 50  0001 C CNN
+F 2 "TO_SOT_Packages_SMD:TO-263-2" H 6800 4400 50  0001 C CNN
 F 3 "" H 6600 4300 50  0001 C CNN
 	1    6600 4300
@@
 F 0 "R1" V 4830 4500 50  0000 C CNN
 F 1 "10k" V 4750 4500 50  0000 C CNN
-F 2 "Resistors_SMD:R_0805_HandSoldering" V 4680 4500 50  0001 C CNN
+F 2 "Resistors_SMD:R_0603_HandSoldering" V 4680 4500 50  0001 C CNN
 F 3 "" H 4750 4500 50  0001 C CNN
 	1    4750 4500
@@
 F 0 "R2" V 6430 4500 50  0000 C CNN
 F 1 "10k" V 6350 4500 50  0000 C CNN
-F 2 "Resistors_SMD:R_0805_HandSoldering" V 6280 4500 50  0001 C CNN
+F 2 "Resistors_SMD:R_0603_HandSoldering" V 6280 4500 50  0001 C CNN
 F 3 "" H 6350 4500 50  0001 C CNN
 	1    6350 4500
@@
 F 0 "J1" H 8350 2500 50  0000 C CNN
 F 1 "Conn_01x16_Male" H 8350 800 50  0000 C CNN
-F 2 "" H 8350 1700 50  0001 C CNN
+F 2 "Connectors_Molex:Molex_MiniFit-JR-5556-16A_2x08x4.20mm_Straight" H 8350 1700 50  0001 C CNN
 F 3 "" H 8350 1700 50  0001 C CNN
 	1    8350 1700
@@
 F 0 "J2" H 8150 3250 50  0000 C CNN
 F 1 "Conn_01x04_Male" H 8150 2750 50  0000 C CNN
-F 2 "" H 8150 3050 50  0001 C CNN
+F 2 "Connectors_Molex:Molex_MiniFit-JR-5556-04A_2x02x4.20mm_Straight" H 8150 3050 50  0001 C CNN
 F 3 "" H 8150 3050 50  0001 C CNN
 	1    8150 3050
@@
 src?
 $Comp
-L Conn_01x05_Male J8
-U 1 1 5A1F5EC6
-P 6600 2450
-F 0 "J8" H 6600 2750 50  0000 C CNN
-F 1 "Conn_01x05_Male" H 6600 2150 50  0000 C CNN
-F 2 "" H 6600 2450 50  0001 C CNN
-F 3 "" H 6600 2450 50  0001 C CNN
-	1    6600 2450
-	-1   0    0    -1
-$EndComp
-$Comp
 L GND #PWR020
 U 1 1 5A1F6F20
-P 6400 2250
-F 0 "#PWR020" H 6400 2000 50  0001 C CNN
-F 1 "GND" H 6400 2100 50  0000 C CNN
-F 2 "" H 6400 2250 50  0001 C CNN
-F 3 "" H 6400 2250 50  0001 C CNN
-	1    6400 2250
-	0    1    1    0
-$EndComp
-NoConn ~ 6400 2350
-NoConn ~ 6400 2450
-NoConn ~ 6400 2650
+P 6700 2150
+F 0 "#PWR020" H 6700 1900 50  0001 C CNN
+F 1 "GND" H 6700 2000 50  0000 C CNN
+F 2 "" H 6700 2150 50  0001 C CNN
+F 3 "" H 6700 2150 50  0001 C CNN
+	1    6700 2150
+	0    1    1    0
+$EndComp
+NoConn ~ 6700 2250
+NoConn ~ 6700 2350
+NoConn ~ 6700 2550
 NoConn ~ 7950 2950
 Text Notes 8750 3200 0    60   ~ 0
@@
 Wire Wire Line
 	3300 3000 3350 3000
+Text Label 5550 6150 2    60   ~ 0
+IMD_RST+
+Text Label 5550 6300 2    60   ~ 0
+IMD_RST-
+$Comp
+L Conn_01x06_Male J8
+U 1 1 5A49ACBF
+P 6900 2350
+F 0 "J8" H 6900 2650 50  0000 C CNN
+F 1 "Conn_01x06_Male" H 6900 1950 50  0000 C CNN
+F 2 "Connectors_Molex:Molex_MiniFit-JR-5556-06A_2x03x4.20mm_Straight" H 6900 2350 50  0001 C CNN
+F 3 "" H 6900 2350 50  0001 C CNN
+	1    6900 2350
+	-1   0    0    -1
+$EndComp
 $EndSCHEMATC
