File: Motherboard.sch (KiCad schematic (older format))
At the start: 34 parts, among them J1 Conn_01x16_Male, J10 Conn_01x01, J11 Conn_01x01, J12 Conn_01x01, J2 Conn_01x04_Male, J3 Conn_01x14_Male, J4 Conn_01x14_Male, J5 Conn_01x14_Male, J8 Conn_01x06_Male, J9 Conn_01x01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

Commit message: final design competition 2018
Parts:
- C18: value C -> 1u
- SW2: footprint TO_SOT_Packages_THT:TO-247_TO-3P_Vertical -> TO_SOT_Packages_THT:TO-220-3_Vertical
Changed lines of the file:
@@
 P 5000 6350
 F 0 "C18" H 5025 6450 50  0000 L CNN
-F 1 "C" H 5025 6250 50  0000 L CNN
+F 1 "1u" H 5025 6250 50  0000 L CNN
 F 2 "Resistors_SMD:R_0805_HandSoldering" H 5038 6200 50  0001 C CNN
 F 3 "" H 5000 6350 50  0001 C CNN
@@
 F 0 "SW2" H 7200 1420 50  0000 C CNN
 F 1 "SW_SPDT" H 7200 1050 50  0000 C CNN
-F 2 "TO_SOT_Packages_THT:TO-247_TO-3P_Vertical" H 7200 1250 50  0001 C CNN
+F 2 "TO_SOT_Packages_THT:TO-220-3_Vertical" H 7200 1250 50  0001 C CNN
 F 3 "" H 7200 1250 50  0001 C CNN
 	1    7200 1250
@@
 Wire Wire Line
 	7550 1300 7400 1350
+Text Label 9850 5550 2    60   ~ 0
+COCKPIT_SW
 $EndSCHEMATC
