File: SignalDelay.sch (KiCad schematic (older format))
At the start: 5 parts, among them U5 NC7WZ17_Schmitt_Trig

Commit message: added noel's revisions
Parts:
- removed U5: NC7WZ17_Schmitt_Trig, symbol NC7WZ17_Schmitt_Trig
- added U?: 74HC14_alt, symbol 74HC14_alt
Connections:
- net labels added: A1', A2'
- wire segments 19 -> 18
Other:
- moved on the sheet: C7, C8, R7, R8
Changed lines of the file:
@@
 $EndDescr
-$Comp
-L NC7WZ17_Schmitt_Trig U5
-U 1 1 5A03445D
-P 4800 3050
-F 0 "U5" H 4650 3100 60  0000 C CNN
-F 1 "NC7WZ17_Schmitt_Trig" H 4750 3200 60  0000 C CNN
-F 2 "" H 4800 3050 60  0001 C CNN
-F 3 "" H 4800 3050 60  0001 C CNN
-	1    4800 3050
-	1    0    0    -1
-$EndComp
 $Comp
 L R R7
 U 1 1 5A0344CB
-P 3450 3150
-F 0 "R7" V 3530 3150 50  0000 C CNN
-F 1 "R" V 3450 3150 50  0000 C CNN
-F 2 "" V 3380 3150 50  0001 C CNN
-F 3 "" H 3450 3150 50  0001 C CNN
-	1    3450 3150
-	0    1    1    0
-$EndComp
-$Comp
-L R R8
-U 1 1 5A034522
 P 3450 3350
-F 0 "R8" V 3530 3350 50  0000 C CNN
+F 0 "R7" V 3530 3350 50  0000 C CNN
 F 1 "R" V 3450 3350 50  0000 C CNN
 F 2 "" V 3380 3350 50  0001 C CNN
@@
 $EndComp
 $Comp
-L +5V #PWR37
+L R R8
+U 1 1 5A034522
+P 3450 3550
+F 0 "R8" V 3530 3550 50  0000 C CNN
+F 1 "R" V 3450 3550 50  0000 C CNN
+F 2 "" V 3380 3550 50  0001 C CNN
+F 3 "" H 3450 3550 50  0001 C CNN
+	1    3450 3550
+	0    1    1    0
+$EndComp
+$Comp
+L +5V #PWR43
 U 1 1 5A0345FB
-P 4000 2750
-F 0 "#PWR37" H 4000 2600 50  0001 C CNN
-F 1 "+5V" H 4000 2890 50  0000 C CNN
-F 2 "" H 4000 2750 50  0001 C CNN
-F 3 "" H 4000 2750 50  0001 C CNN
-	1    4000 2750
+P 4200 3750
+F 0 "#PWR43" H 4200 3600 50  0001 C CNN
+F 1 "+5V" H 4200 3890 50  0000 C CNN
+F 2 "" H 4200 3750 50  0001 C CNN
+F 3 "" H 4200 3750 50  0001 C CNN
+	1    4200 3750
 	1    0    0    -1
 $EndComp
@@
 L CP C7
 U 1 1 5A03464B
-P 3650 3650
-F 0 "C7" H 3675 3750 50  0000 L CNN
-F 1 "CP" H 3675 3550 50  0000 L CNN
-F 2 "" H 3688 3500 50  0001 C CNN
-F 3 "" H 3650 3650 50  0001 C CNN
-	1    3650 3650
+P 3650 3850
+F 0 "C7" H 3675 3950 50  0000 L CNN
+F 1 "CP" H 3675 3750 50  0000 L CNN
+F 2 "" H 3688 3700 50  0001 C CNN
+F 3 "" H 3650 3850 50  0001 C CNN
+	1    3650 3850
 	1    0    0    -1
 $EndComp
@@
 L CP C8
 U 1 1 5A034698
-P 3900 3650
-F 0 "C8" H 3925 3750 50  0000 L CNN
-F 1 "CP" H 3925 3550 50  0000 L CNN
-F 2 "" H 3938 3500 50  0001 C CNN
-F 3 "" H 3900 3650 50  0001 C CNN
-	1    3900 3650
+P 3900 3850
+F 0 "C8" H 3925 3950 50  0000 L CNN
+F 1 "CP" H 3925 3750 50  0000 L CNN
+F 2 "" H 3938 3700 50  0001 C CNN
+F 3 "" H 3900 3850 50  0001 C CNN
+	1    3900 3850
 	1    0    0    -1
 $EndComp
 $Comp
-L GND #PWR36
+L GND #PWR42
 U 1 1 5A03473A
-P 3900 4000
-F 0 "#PWR36" H 3900 3750 50  0001 C CNN
-F 1 "GND" H 3900 3850 50  0000 C CNN
-F 2 "" H 3900 4000 50  0001 C CNN
-F 3 "" H 3900 4000 50  0001 C CNN
-	1    3900 4000
+P 3650 4300
+F 0 "#PWR42" H 3650 4050 50  0001 C CNN
+F 1 "GND" H 3650 4150 50  0000 C CNN
+F 2 "" H 3650 4300 50  0001 C CNN
+F 3 "" H 3650 4300 50  0001 C CNN
+	1    3650 4300
 	1    0    0    -1
 $EndComp
-Text HLabel 3100 3150 0    60   Input ~ 0
+Text HLabel 4350 3150 0    60   Input ~ 0
 A1
-Text HLabel 3100 3350 0    60   Input ~ 0
+Text HLabel 4350 3250 0    60   Input ~ 0
 A2
 Wire Wire Line
-	3600 3150 4350 3150
+	3600 3350 4350 3350
 Wire Wire Line
-	3600 3350 4200 3350
+	3600 3550 4200 3550
 Wire Wire Line
-	4200 3350 4200 3250
+	3650 3350 3650 3700
 Wire Wire Line
-	4200 3250 4350 3250
+	3900 3700 3900 3550
+Connection ~ 3900 3550
 Wire Wire Line
-	4350 3450 4000 3450
+	3650 4000 3650 4300
 Wire Wire Line
-	4000 3450 4000 2750
-Wire Wire Line
-	3650 3500 3650 3150
-Connection ~ 3650 3150
-Wire Wire Line
-	3900 3500 3900 3350
-Connection ~ 3900 3350
-Wire Wire Line
-	3650 3800 3650 3900
-Wire Wire Line
-	3650 3900 5400 3900
-Wire Wire Line
-	3900 3800 3900 4000
-Connection ~ 3900 3900
-Wire Wire Line
-	3300 3150 3100 3150
+	3900 4000 3900 4200
 Wire Wire Line
 	3300 3350 3100 3350
 Wire Wire Line
-	5250 3150 5700 3150
+	3300 3550 3100 3550
 Wire Wire Line
-	5250 3250 5450 3250
+	5250 3350 5700 3350
 Wire Wire Line
-	5450 3250 5450 3350
+	5250 3450 5450 3450
 Wire Wire Line
-	5450 3350 5700 3350
-Text HLabel 5700 3150 2    60   Output ~ 0
+	5450 3450 5450 3550
+Wire Wire Line
+	5450 3550 5700 3550
+Text HLabel 5700 3350 2    60   Output ~ 0
 Y1
-Text HLabel 5700 3350 2    60   Output ~ 0
+Text HLabel 5700 3550 2    60   Output ~ 0
 Y2
+$Comp
+L 74HC14_alt U?
+U 1 1 5A112856
+P 4800 3050
+F 0 "U?" H 4650 3100 60  0000 C CNN
+F 1 "74HC14_alt" H 4750 3200 60  0000 C CNN
+F 2 "" H 4800 3050 60  0001 C CNN
+F 3 "" H 4800 3050 60  0001 C CNN
+	1    4800 3050
+	1    0    0    -1
+$EndComp
 Wire Wire Line
-	5250 3450 5400 3450
+	5250 4200 5250 3850
+Text Label 5250 3150 0    60   ~ 0
+A1'
+Text Label 5250 3250 0    60   ~ 0
+A2'
+Text Label 3100 3350 2    60   ~ 0
+A1'
+Text Label 3100 3550 2    60   ~ 0
+A2'
 Wire Wire Line
-	5400 3450 5400 3900
+	4200 3550 4200 3450
+Wire Wire Line
+	4200 3450 4350 3450
+Connection ~ 3650 3350
+Wire Wire Line
+	4200 3750 4200 3850
+Wire Wire Line
+	4200 3850 4350 3850
+Wire Wire Line
+	3650 4200 5250 4200
+Connection ~ 3650 4200
+Connection ~ 3900 4200
 $EndSCHEMATC

Commit message: added charger sd logic
Parts:
- removed U?: 74HC14_alt, symbol 74HC14_alt
- added U? (x4): 74HC14, symbol 74HC14
Connections:
- net labels removed: +5V, A1', A2'
- wire segments 18 -> 14
Other:
- moved on the sheet: C7, C8, R8
Changed lines of the file:
@@
 L R R8
 U 1 1 5A034522
-P 3450 3550
-F 0 "R8" V 3530 3550 50  0000 C CNN
-F 1 "R" V 3450 3550 50  0000 C CNN
-F 2 "" V 3380 3550 50  0001 C CNN
-F 3 "" H 3450 3550 50  0001 C CNN
-	1    3450 3550
+P 3450 3850
+F 0 "R8" V 3530 3850 50  0000 C CNN
+F 1 "R" V 3450 3850 50  0000 C CNN
+F 2 "" V 3380 3850 50  0001 C CNN
+F 3 "" H 3450 3850 50  0001 C CNN
+	1    3450 3850
 	0    1    1    0
-$EndComp
-$Comp
-L +5V #PWR43
-U 1 1 5A0345FB
-P 4200 3750
-F 0 "#PWR43" H 4200 3600 50  0001 C CNN
-F 1 "+5V" H 4200 3890 50  0000 C CNN
-F 2 "" H 4200 3750 50  0001 C CNN
-F 3 "" H 4200 3750 50  0001 C CNN
-	1    4200 3750
-	1    0    0    -1
 $EndComp
 $Comp
 L CP C7
 U 1 1 5A03464B
-P 3650 3850
-F 0 "C7" H 3675 3950 50  0000 L CNN
-F 1 "CP" H 3675 3750 50  0000 L CNN
-F 2 "" H 3688 3700 50  0001 C CNN
-F 3 "" H 3650 3850 50  0001 C CNN
-	1    3650 3850
+P 3650 4150
+F 0 "C7" H 3675 4250 50  0000 L CNN
+F 1 "CP" H 3675 4050 50  0000 L CNN
+F 2 "" H 3688 4000 50  0001 C CNN
+F 3 "" H 3650 4150 50  0001 C CNN
+	1    3650 4150
 	1    0    0    -1
 $EndComp
@@
 L CP C8
 U 1 1 5A034698
-P 3900 3850
-F 0 "C8" H 3925 3950 50  0000 L CNN
-F 1 "CP" H 3925 3750 50  0000 L CNN
-F 2 "" H 3938 3700 50  0001 C CNN
-F 3 "" H 3900 3850 50  0001 C CNN
-	1    3900 3850
+P 3900 4150
+F 0 "C8" H 3925 4250 50  0000 L CNN
+F 1 "CP" H 3925 4050 50  0000 L CNN
+F 2 "" H 3938 4000 50  0001 C CNN
+F 3 "" H 3900 4150 50  0001 C CNN
+	1    3900 4150
 	1    0    0    -1
 $EndComp
@@
 L GND #PWR42
 U 1 1 5A03473A
-P 3650 4300
-F 0 "#PWR42" H 3650 4050 50  0001 C CNN
-F 1 "GND" H 3650 4150 50  0000 C CNN
-F 2 "" H 3650 4300 50  0001 C CNN
-F 3 "" H 3650 4300 50  0001 C CNN
-	1    3650 4300
+P 3650 4600
+F 0 "#PWR42" H 3650 4350 50  0001 C CNN
+F 1 "GND" H 3650 4450 50  0000 C CNN
+F 2 "" H 3650 4600 50  0001 C CNN
+F 3 "" H 3650 4600 50  0001 C CNN
+	1    3650 4600
 	1    0    0    -1
 $EndComp
-Text HLabel 4350 3150 0    60   Input ~ 0
+Text HLabel 2200 3350 0    60   Input ~ 0
 A1
-Text HLabel 4350 3250 0    60   Input ~ 0
+Text HLabel 2200 3850 0    60   Input ~ 0
 A2
 Wire Wire Line
-	3600 3350 4350 3350
+	3600 3850 3900 3850
 Wire Wire Line
-	3600 3550 4200 3550
+	3900 3850 4350 3850
 Wire Wire Line
-	3650 3350 3650 3700
+	3650 3350 3650 4000
 Wire Wire Line
-	3900 3700 3900 3550
-Connection ~ 3900 3550
+	3900 4000 3900 3850
+Connection ~ 3900 3850
 Wire Wire Line
-	3650 4000 3650 4300
+	3650 4300 3650 4500
 Wire Wire Line
-	3900 4000 3900 4200
+	3650 4500 3650 4600
+Wire Wire Line
+	3900 4300 3900 4500
 Wire Wire Line
 	3300 3350 3100 3350
 Wire Wire Line
-	3300 3550 3100 3550
+	3300 3850 3100 3850
 Wire Wire Line
 	5250 3350 5700 3350
 Wire Wire Line
-	5250 3450 5450 3450
-Wire Wire Line
-	5450 3450 5450 3550
-Wire Wire Line
-	5450 3550 5700 3550
+	5250 3850 5700 3850
 Text HLabel 5700 3350 2    60   Output ~ 0
 Y1
-Text HLabel 5700 3550 2    60   Output ~ 0
+Text HLabel 5700 3850 2    60   Output ~ 0
 Y2
+Wire Wire Line
+	3650 4500 3900 4500
+Connection ~ 3650 4500
 $Comp
-L 74HC14_alt U?
-U 1 1 5A112856
-P 4800 3050
-F 0 "U?" H 4650 3100 60  0000 C CNN
-F 1 "74HC14_alt" H 4750 3200 60  0000 C CNN
-F 2 "" H 4800 3050 60  0001 C CNN
-F 3 "" H 4800 3050 60  0001 C CNN
-	1    4800 3050
+L 74HC14 U?
+U 1 1 5A122AA0
+P 2650 3350
+F 0 "U?" H 2800 3450 50  0000 C CNN
+F 1 "74HC14" H 2850 3250 50  0000 C CNN
+F 2 "" H 2650 3350 50  0001 C CNN
+F 3 "" H 2650 3350 50  0001 C CNN
+	1    2650 3350
+	1    0    0    -1
+$EndComp
+$Comp
+L 74HC14 U?
+U 2 1 5A122B13
+P 2650 3850
+F 0 "U?" H 2800 3950 50  0000 C CNN
+F 1 "74HC14" H 2850 3750 50  0000 C CNN
+F 2 "" H 2650 3850 50  0001 C CNN
+F 3 "" H 2650 3850 50  0001 C CNN
+	2    2650 3850
+	1    0    0    -1
+$EndComp
+$Comp
+L 74HC14 U?
+U 3 1 5A122C1C
+P 4800 3350
+F 0 "U?" H 4950 3450 50  0000 C CNN
+F 1 "74HC14" H 5000 3250 50  0000 C CNN
+F 2 "" H 4800 3350 50  0001 C CNN
+F 3 "" H 4800 3350 50  0001 C CNN
+	3    4800 3350
 	1    0    0    -1
 $EndComp
 Wire Wire Line
-	5250 4200 5250 3850
-Text Label 5250 3150 0    60   ~ 0
-A1'
-Text Label 5250 3250 0    60   ~ 0
-A2'
-Text Label 3100 3350 2    60   ~ 0
-A1'
-Text Label 3100 3550 2    60   ~ 0
-A2'
+	3600 3350 3650 3350
 Wire Wire Line
-	4200 3550 4200 3450
-Wire Wire Line
-	4200 3450 4350 3450
+	3650 3350 4350 3350
 Connection ~ 3650 3350
-Wire Wire Line
-	4200 3750 4200 3850
-Wire Wire Line
-	4200 3850 4350 3850
-Wire Wire Line
-	3650 4200 5250 4200
-Connection ~ 3650 4200
-Connection ~ 3900 4200
+$Comp
+L 74HC14 U?
+U 4 1 5A122D66
+P 4800 3850
+F 0 "U?" H 4950 3950 50  0000 C CNN
+F 1 "74HC14" H 5000 3750 50  0000 C CNN
+F 2 "" H 4800 3850 50  0001 C CNN
+F 3 "" H 4800 3850 50  0001 C CNN
+	4    4800 3850
+	1    0    0    -1
+$EndComp
 $EndSCHEMATC
