File: SignalDelay.sch (KiCad schematic (older format))
At the start: 5 parts, among them U6 74HC14

Commit message: beginning board design
Parts:
- U6: footprint (none) -> Housings_DIP:DIP-14_W8.89mm_SMDSocket_LongPads
- renumbered R9 to R7, R10 to R8
Changed lines of the file:
@@
 $EndDescr
 $Comp
-L R R9
+L R R7
 U 1 1 5A0344CB
 P 3450 3350
-F 0 "R9" V 3530 3350 50  0000 C CNN
+F 0 "R7" V 3530 3350 50  0000 C CNN
 F 1 "R" V 3450 3350 50  0000 C CNN
 F 2 "" V 3380 3350 50  0001 C CNN
@@
 $EndComp
 $Comp
-L R R10
+L R R8
 U 1 1 5A034522
 P 3450 3850
-F 0 "R10" V 3530 3850 50  0000 C CNN
+F 0 "R8" V 3530 3850 50  0000 C CNN
 F 1 "R" V 3450 3850 50  0000 C CNN
 F 2 "" V 3380 3850 50  0001 C CNN
@@
 $EndComp
 $Comp
-L GND #PWR39
+L GND #PWR037
 U 1 1 5A03473A
 P 3650 4600
-F 0 "#PWR39" H 3650 4350 50  0001 C CNN
+F 0 "#PWR037" H 3650 4350 50  0001 C CNN
 F 1 "GND" H 3650 4450 50  0000 C CNN
 F 2 "" H 3650 4600 50  0001 C CNN
@@
 F 0 "U6" H 2800 3450 50  0000 C CNN
 F 1 "74HC14" H 2850 3250 50  0000 C CNN
-F 2 "" H 2650 3350 50  0001 C CNN
+F 2 "Housings_DIP:DIP-14_W8.89mm_SMDSocket_LongPads" H 2650 3350 50  0001 C CNN
 F 3 "" H 2650 3350 50  0001 C CNN
 	1    2650 3350
@@
 F 0 "U6" H 2800 3950 50  0000 C CNN
 F 1 "74HC14" H 2850 3750 50  0000 C CNN
-F 2 "" H 2650 3850 50  0001 C CNN
+F 2 "Housings_DIP:DIP-14_W8.89mm_SMDSocket_LongPads" H 2650 3850 50  0001 C CNN
 F 3 "" H 2650 3850 50  0001 C CNN
 	2    2650 3850
@@
 F 0 "U6" H 4950 3450 50  0000 C CNN
 F 1 "74HC14" H 5000 3250 50  0000 C CNN
-F 2 "" H 4800 3350 50  0001 C CNN
+F 2 "Housings_DIP:DIP-14_W8.89mm_SMDSocket_LongPads" H 4800 3350 50  0001 C CNN
 F 3 "" H 4800 3350 50  0001 C CNN
 	3    4800 3350
@@
 F 0 "U6" H 4950 3950 50  0000 C CNN
 F 1 "74HC14" H 5000 3750 50  0000 C CNN
-F 2 "" H 4800 3850 50  0001 C CNN
+F 2 "Housings_DIP:DIP-14_W8.89mm_SMDSocket_LongPads" H 4800 3850 50  0001 C CNN
 F 3 "" H 4800 3850 50  0001 C CNN
 	4    4800 3850

Commit message: beginning floorplan
Connections:
- net labels added: +5V
Changed lines of the file:
@@
 $EndComp
 $Comp
-L GND #PWR39
+L GND #PWR040
 U 1 1 5A03473A
 P 3650 4600
-F 0 "#PWR39" H 3650 4350 50  0001 C CNN
+F 0 "#PWR040" H 3650 4350 50  0001 C CNN
 F 1 "GND" H 3650 4450 50  0000 C CNN
 F 2 "" H 3650 4600 50  0001 C CNN
@@
 	1    0    0    -1
 $EndComp
+$Comp
+L +5V #PWR041
+U 1 1 5A2BEB33
+P 2600 3250
+F 0 "#PWR041" H 2600 3100 50  0001 C CNN
+F 1 "+5V" H 2600 3390 50  0000 C CNN
+F 2 "" H 2600 3250 50  0001 C CNN
+F 3 "" H 2600 3250 50  0001 C CNN
+	1    2600 3250
+	1    0    0    -1
+$EndComp

Commit message: winter break changes
Parts:
- C7, C8: footprint (none) -> Capacitors_THT:CP_Radial_D8.0mm_P5.00mm
- R7, R8: footprint (none) -> Resistors_SMD:R_0603_HandSoldering
Changed lines of the file:
@@
 F 0 "R7" V 3530 3350 50  0000 C CNN
 F 1 "R" V 3450 3350 50  0000 C CNN
-F 2 "" V 3380 3350 50  0001 C CNN
+F 2 "Resistors_SMD:R_0603_HandSoldering" V 3380 3350 50  0001 C CNN
 F 3 "" H 3450 3350 50  0001 C CNN
 	1    3450 3350
@@
 F 0 "R8" V 3530 3850 50  0000 C CNN
 F 1 "R" V 3450 3850 50  0000 C CNN
-F 2 "" V 3380 3850 50  0001 C CNN
+F 2 "Resistors_SMD:R_0603_HandSoldering" V 3380 3850 50  0001 C CNN
 F 3 "" H 3450 3850 50  0001 C CNN
 	1    3450 3850
@@
 F 0 "C7" H 3675 4250 50  0000 L CNN
 F 1 "CP" H 3675 4050 50  0000 L CNN
-F 2 "" H 3688 4000 50  0001 C CNN
+F 2 "Capacitors_THT:CP_Radial_D8.0mm_P5.00mm" H 3688 4000 50  0001 C CNN
 F 3 "" H 3650 4150 50  0001 C CNN
 	1    3650 4150
@@
 F 0 "C8" H 3925 4250 50  0000 L CNN
 F 1 "CP" H 3925 4050 50  0000 L CNN
-F 2 "" H 3938 4000 50  0001 C CNN
+F 2 "Capacitors_THT:CP_Radial_D8.0mm_P5.00mm" H 3938 4000 50  0001 C CNN
 F 3 "" H 3900 4150 50  0001 C CNN
 	1    3900 4150

Commit message: finished routing
Parts:
- removed C7, C8: CP, Capacitors_THT:CP_Radial_D8.0mm_P5.00mm, symbol CP
- added C13, C14, C7, C8: C, Capacitors_SMD:C_0805_HandSoldering, symbol C
- R7, R8: footprint Resistors_SMD:R_0603_HandSoldering -> Resistors_SMD:R_0805_HandSoldering
Connections:
- wire segments 11 -> 17
Changed lines of the file:
@@
 F 0 "R7" V 3530 3350 50  0000 C CNN
 F 1 "R" V 3450 3350 50  0000 C CNN
-F 2 "Resistors_SMD:R_0603_HandSoldering" V 3380 3350 50  0001 C CNN
+F 2 "Resistors_SMD:R_0805_HandSoldering" V 3380 3350 50  0001 C CNN
 F 3 "" H 3450 3350 50  0001 C CNN
 	1    3450 3350
@@
 F 0 "R8" V 3530 3850 50  0000 C CNN
 F 1 "R" V 3450 3850 50  0000 C CNN
-F 2 "Resistors_SMD:R_0603_HandSoldering" V 3380 3850 50  0001 C CNN
+F 2 "Resistors_SMD:R_0805_HandSoldering" V 3380 3850 50  0001 C CNN
 F 3 "" H 3450 3850 50  0001 C CNN
 	1    3450 3850
@@
 $EndComp
 $Comp
-L CP C7
-U 1 1 5A03464B
-P 3650 4150
-F 0 "C7" H 3675 4250 50  0000 L CNN
-F 1 "CP" H 3675 4050 50  0000 L CNN
-F 2 "Capacitors_THT:CP_Radial_D8.0mm_P5.00mm" H 3688 4000 50  0001 C CNN
-F 3 "" H 3650 4150 50  0001 C CNN
-	1    3650 4150
-	1    0    0    -1
-$EndComp
-$Comp
-L CP C8
-U 1 1 5A034698
-P 3900 4150
-F 0 "C8" H 3925 4250 50  0000 L CNN
-F 1 "CP" H 3925 4050 50  0000 L CNN
-F 2 "Capacitors_THT:CP_Radial_D8.0mm_P5.00mm" H 3938 4000 50  0001 C CNN
-F 3 "" H 3900 4150 50  0001 C CNN
-	1    3900 4150
-	1    0    0    -1
-$EndComp
-$Comp
-L GND #PWR040
+L GND #PWR048
 U 1 1 5A03473A
 P 3650 4600
-F 0 "#PWR040" H 3650 4350 50  0001 C CNN
+F 0 "#PWR048" H 3650 4350 50  0001 C CNN
 F 1 "GND" H 3650 4450 50  0000 C CNN
 F 2 "" H 3650 4600 50  0001 C CNN
@@
 	3650 4300 3650 4600
 Wire Wire Line
-	3900 4300 3900 4500
+	3900 4500 3900 4300
 Wire Wire Line
 	3300 3350 3100 3350
@@
 Y2
 Wire Wire Line
-	3900 4500 3650 4500
+	3400 4500 4150 4500
 Connection ~ 3650 4500
 $Comp
@@
 $EndComp
 $Comp
-L +5V #PWR041
+L +5V #PWR049
 U 1 1 5A2BEB33
 P 2600 3250
-F 0 "#PWR041" H 2600 3100 50  0001 C CNN
+F 0 "#PWR049" H 2600 3100 50  0001 C CNN
 F 1 "+5V" H 2600 3390 50  0000 C CNN
 F 2 "" H 2600 3250 50  0001 C CNN
@@
 	1    0    0    -1
 $EndComp
+$Comp
+L C C13
+U 1 1 5A679E7D
+P 3900 4150
+F 0 "C13" H 3925 4250 50  0000 L CNN
+F 1 "C" H 3925 4050 50  0000 L CNN
+F 2 "Capacitors_SMD:C_0805_HandSoldering" H 3938 4000 50  0001 C CNN
+F 3 "" H 3900 4150 50  0001 C CNN
+	1    3900 4150
+	1    0    0    -1
+$EndComp
+$Comp
+L C C14
+U 1 1 5A679EC1
+P 4150 4150
+F 0 "C14" H 4175 4250 50  0000 L CNN
+F 1 "C" H 4175 4050 50  0000 L CNN
+F 2 "Capacitors_SMD:C_0805_HandSoldering" H 4188 4000 50  0001 C CNN
+F 3 "" H 4150 4150 50  0001 C CNN
+	1    4150 4150
+	1    0    0    -1
+$EndComp
+$Comp
+L C C8
+U 1 1 5A679EEF
+P 3650 4150
+F 0 "C8" H 3675 4250 50  0000 L CNN
+F 1 "C" H 3675 4050 50  0000 L CNN
+F 2 "Capacitors_SMD:C_0805_HandSoldering" H 3688 4000 50  0001 C CNN
+F 3 "" H 3650 4150 50  0001 C CNN
+	1    3650 4150
+	1    0    0    -1
+$EndComp
+$Comp
+L C C7
+U 1 1 5A679F2A
+P 3400 4150
+F 0 "C7" H 3425 4250 50  0000 L CNN
+F 1 "C" H 3425 4050 50  0000 L CNN
+F 2 "Capacitors_SMD:C_0805_HandSoldering" H 3438 4000 50  0001 C CNN
+F 3 "" H 3400 4150 50  0001 C CNN
+	1    3400 4150
+	1    0    0    -1
+$EndComp
+Wire Wire Line
+	3400 4000 3400 3950
+Wire Wire Line
+	3400 3950 3650 3950
+Connection ~ 3650 3950
+Wire Wire Line
+	3400 4300 3400 4500
+Wire Wire Line
+	3900 3950 4150 3950
+Wire Wire Line
+	4150 3950 4150 4000
+Connection ~ 3900 3950
+Wire Wire Line
+	4150 4500 4150 4300
+Connection ~ 3900 4500
 $EndSCHEMATC
