File: _saved_ShutdownCircuit.sch (KiCad schematic (older format))
At the start: 12 parts, among them K1 IMD_RELAY, K2 IMD_LATCH, K3 BMS_RELAY, Q3 Q_NMOS_DGS, Q4 Q_NMOS_DGS

Commit message: added most footprint associations
Parts:
- D1: value LED -> IMD_OK
- D2: footprint (none) -> Diodes_SMD:D_0805
- D3: value LED -> BMS_OK
- renumbered F12 to F13, R5 to R10, R4 to R9
Changed lines of the file:
@@
 $EndDescr
 $Comp
-L +12V #PWR17
+L +12V #PWR038
 U 1 1 5A022276
 P 2900 2150
-F 0 "#PWR17" H 2900 2000 50  0001 C CNN
+F 0 "#PWR038" H 2900 2000 50  0001 C CNN
 F 1 "+12V" H 2900 2290 50  0000 C CNN
 F 2 "" H 2900 2150 50  0001 C CNN
@@
 $EndComp
 $Comp
-L +12V #PWR18
+L +12V #PWR039
 U 1 1 5A02229A
 P 3050 3350
-F 0 "#PWR18" H 3050 3200 50  0001 C CNN
+F 0 "#PWR039" H 3050 3200 50  0001 C CNN
 F 1 "+12V" H 3050 3490 50  0000 C CNN
 F 2 "" H 3050 3350 50  0001 C CNN
@@
 $EndComp
 $Comp
-L +12V #PWR20
+L +12V #PWR040
 U 1 1 5A0222EA
 P 5250 2550
-F 0 "#PWR20" H 5250 2400 50  0001 C CNN
+F 0 "#PWR040" H 5250 2400 50  0001 C CNN
 F 1 "+12V" H 5250 2690 50  0000 C CNN
 F 2 "" H 5250 2550 50  0001 C CNN
@@
 F 0 "D2" H 4300 4350 50  0000 C CNN
 F 1 "IMD_FLYBACK" H 4300 4150 50  0000 C CNN
-F 2 "" H 4300 4250 50  0001 C CNN
+F 2 "Diodes_SMD:D_0805" H 4300 4250 50  0001 C CNN
 F 3 "" H 4300 4250 50  0001 C CNN
 	1    4300 4250
@@
 $EndComp
 $Comp
-L GND #PWR19
+L GND #PWR041
 U 1 1 5A022431
 P 4850 5250
-F 0 "#PWR19" H 4850 5000 50  0001 C CNN
+F 0 "#PWR041" H 4850 5000 50  0001 C CNN
 F 1 "GND" H 4850 5100 50  0000 C CNN
 F 2 "" H 4850 5250 50  0001 C CNN
@@
 P 4100 4550
 F 0 "D1" H 4100 4650 50  0000 C CNN
-F 1 "LED" H 4100 4450 50  0000 C CNN
+F 1 "IMD_OK" H 4100 4450 50  0000 C CNN
 F 2 "" H 4100 4550 50  0001 C CNN
 F 3 "" H 4100 4550 50  0001 C CNN
@@
 $EndComp
 $Comp
-L R R4
+L R R9
 U 1 1 5A09EADD
 P 4550 4550
-F 0 "R4" V 4630 4550 50  0000 C CNN
+F 0 "R9" V 4630 4550 50  0000 C CNN
 F 1 "R" V 4550 4550 50  0000 C CNN
 F 2 "" V 4480 4550 50  0001 C CNN
@@
 P 5600 3300
 F 0 "D3" H 5600 3400 50  0000 C CNN
-F 1 "LED" H 5600 3200 50  0000 C CNN
+F 1 "BMS_OK" H 5600 3200 50  0000 C CNN
 F 2 "" H 5600 3300 50  0001 C CNN
 F 3 "" H 5600 3300 50  0001 C CNN
@@
 $EndComp
 $Comp
-L R R5
+L R R10
 U 1 1 5A09ED01
 P 6050 3300
-F 0 "R5" V 6130 3300 50  0000 C CNN
+F 0 "R10" V 6130 3300 50  0000 C CNN
 F 1 "R" V 6050 3300 50  0000 C CNN
 F 2 "" V 5980 3300 50  0001 C CNN
@@
 Connection ~ 6350 2950
 $Comp
-L Fuse F12
+L Fuse F13
 U 1 1 5A122E62
 P 3500 2150
-F 0 "F12" V 3580 2150 50  0000 C CNN
+F 0 "F13" V 3580 2150 50  0000 C CNN
 F 1 "SD_FUSE" V 3425 2150 50  0000 C CNN
 F 2 "" V 3430 2150 50  0001 C CNN
