File: _saved_SignalDelay.sch (KiCad schematic (older format))
At the start: 5 parts, among them U6 74HC14

Commit message: added most footprint associations
Parts:
- renumbered R9 to R7, R10 to R8
Changed lines of the file:
@@
 $EndDescr
 $Comp
-L R R9
+L R R7
 U 1 1 5A0344CB
 P 3450 3350
-F 0 "R9" V 3530 3350 50  0000 C CNN
+F 0 "R7" V 3530 3350 50  0000 C CNN
 F 1 "R" V 3450 3350 50  0000 C CNN
 F 2 "" V 3380 3350 50  0001 C CNN
@@
 $EndComp
 $Comp
-L R R10
+L R R8
 U 1 1 5A034522
 P 3450 3850
-F 0 "R10" V 3530 3850 50  0000 C CNN
+F 0 "R8" V 3530 3850 50  0000 C CNN
 F 1 "R" V 3450 3850 50  0000 C CNN
 F 2 "" V 3380 3850 50  0001 C CNN
@@
 $EndComp
 $Comp
-L GND #PWR39
+L GND #PWR037
 U 1 1 5A03473A
 P 3650 4600
-F 0 "#PWR39" H 3650 4350 50  0001 C CNN
+F 0 "#PWR037" H 3650 4350 50  0001 C CNN
 F 1 "GND" H 3650 4450 50  0000 C CNN
 F 2 "" H 3650 4600 50  0001 C CNN
