File: _saved_Motherboard.sch (KiCad schematic (older format))
At the start: 34 parts, among them J1 Conn_01x16_Male, J10 Conn_01x01, J11 Conn_01x01, J12 Conn_01x01, J2 Conn_01x04_Male, J3 Conn_01x14_Male, J4 Conn_01x14_Male, J5 Conn_01x14_Male, J8 Conn_01x06_Male, J9 Conn_01x01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

Commit message: finished routing
Parts:
- SW2: footprint TO_SOT_Packages_THT:TO-247_TO-3P_Vertical -> TO_SOT_Packages_THT:TO-220-3_Vertical
Changed lines of the file:
@@
 F 0 "SW2" H 7200 1420 50  0000 C CNN
 F 1 "SW_SPDT" H 7200 1050 50  0000 C CNN
-F 2 "TO_SOT_Packages_THT:TO-247_TO-3P_Vertical" H 7200 1250 50  0001 C CNN
+F 2 "TO_SOT_Packages_THT:TO-220-3_Vertical" H 7200 1250 50  0001 C CNN
 F 3 "" H 7200 1250 50  0001 C CNN
 	1    7200 1250
