File: Logic.sch (KiCad schematic (older format))
At the start: 15 parts, among them J1 FTDI, J2 ICSP, SW2 SW_Push, U2 CD4050, U3 ATMEGA328P-MU, U4 CD40109

Commit message: added noel's revisions
Parts:
- removed U3: ATMEGA328P-MU, MLF/QFN32, symbol ATMEGA328P-MU
- added U?: ATMEGA328P-PU, DIL28, symbol ATMEGA328P-PU
Connections:
- net labels added: TSMS
- net labels removed: CONTACT_REQ
- wire segments 82 -> 80
- no-connect marks 2 -> 6
Changed lines of the file:
@@
 $EndDescr
 $Comp
-L ATMEGA328P-MU U3
-U 1 1 5A0238D6
-P 4400 4500
-F 0 "U3" H 3650 5750 50  0000 L BNN
-F 1 "ATMEGA328P-MU" H 4800 3100 50  0000 L BNN
-F 2 "MLF/QFN32" H 4400 4500 50  0001 C CIN
-F 3 "" H 4400 4500 50  0001 C CNN
-	1    4400 4500
-	1    0    0    -1
-$EndComp
-$Comp
-L +5V #PWR18
+L +5V #PWR24
 U 1 1 5A023903
 P 3050 3300
-F 0 "#PWR18" H 3050 3150 50  0001 C CNN
+F 0 "#PWR24" H 3050 3150 50  0001 C CNN
 F 1 "+5V" H 3050 3440 50  0000 C CNN
 F 2 "" H 3050 3300 50  0001 C CNN
@@
 $EndComp
 $Comp
-L GND #PWR19
+L GND #PWR25
 U 1 1 5A0239BE
 P 3050 4150
-F 0 "#PWR19" H 3050 3900 50  0001 C CNN
+F 0 "#PWR25" H 3050 3900 50  0001 C CNN
 F 1 "GND" H 3050 4000 50  0000 C CNN
 F 2 "" H 3050 4150 50  0001 C CNN
@@
 $EndComp
 $Comp
-L GND #PWR21
+L GND #PWR27
 U 1 1 5A023B6E
 P 3400 5850
-F 0 "#PWR21" H 3400 5600 50  0001 C CNN
+F 0 "#PWR27" H 3400 5600 50  0001 C CNN
 F 1 "GND" H 3400 5700 50  0000 C CNN
 F 2 "" H 3400 5850 50  0001 C CNN
@@
 TSMS_12V
 $Comp
-L GND #PWR23
+L GND #PWR29
 U 1 1 5A024854
 P 4750 1400
-F 0 "#PWR23" H 4750 1150 50  0001 C CNN
+F 0 "#PWR29" H 4750 1150 50  0001 C CNN
 F 1 "GND" H 4750 1250 50  0000 C CNN
 F 2 "" H 4750 1400 50  0001 C CNN
@@
 $EndComp
 $Comp
-L +12V #PWR22
+L +12V #PWR28
 U 1 1 5A024870
 P 3500 1050
-F 0 "#PWR22" H 3500 900 50  0001 C CNN
+F 0 "#PWR28" H 3500 900 50  0001 C CNN
 F 1 "+12V" H 3500 1190 50  0000 C CNN
 F 2 "" H 3500 1050 50  0001 C CNN
@@
 BOTS
 Text Label 5400 5700 0    60   ~ 0
-TSMS_12V
-Text Label 5400 3600 0    60   ~ 0
-CONTACT_REQ
+TSMS
 $Comp
 L CD40109 U4
@@
 BOTS
 Text Label 4500 2300 0    60   ~ 0
-TSMS_12V
-$Comp
-L +12V #PWR25
+TSMS
+$Comp
+L +12V #PWR31
 U 1 1 5A0259BE
 P 6350 2600
-F 0 "#PWR25" H 6350 2450 50  0001 C CNN
+F 0 "#PWR31" H 6350 2450 50  0001 C CNN
 F 1 "+12V" H 6350 2740 50  0000 C CNN
 F 2 "" H 6350 2600 50  0001 C CNN
@@
 $EndComp
 $Comp
-L +5V #PWR30
+L +5V #PWR36
 U 1 1 5A0259DC
 P 6800 2250
-F 0 "#PWR30" H 6800 2100 50  0001 C CNN
+F 0 "#PWR36" H 6800 2100 50  0001 C CNN
 F 1 "+5V" H 6800 2390 50  0000 C CNN
 F 2 "" H 6800 2250 50  0001 C CNN
@@
 $EndComp
 $Comp
-L GND #PWR33
+L GND #PWR39
 U 1 1 5A025A80
 P 8000 2650
-F 0 "#PWR33" H 8000 2400 50  0001 C CNN
+F 0 "#PWR39" H 8000 2400 50  0001 C CNN
 F 1 "GND" H 8000 2500 50  0000 C CNN
 F 2 "" H 8000 2650 50  0001 C CNN
@@
 $EndComp
 $Comp
-L +5V #PWR32
+L +5V #PWR38
 U 1 1 5A025B81
 P 8000 2250
-F 0 "#PWR32" H 8000 2100 50  0001 C CNN
+F 0 "#PWR38" H 8000 2100 50  0001 C CNN
 F 1 "+5V" H 8000 2390 50  0000 C CNN
 F 2 "" H 8000 2250 50  0001 C CNN
@@
 $EndComp
 $Comp
-L +5V #PWR24
+L +5V #PWR30
 U 1 1 5A02647A
 P 6200 4200
-F 0 "#PWR24" H 6200 4050 50  0001 C CNN
+F 0 "#PWR30" H 6200 4050 50  0001 C CNN
 F 1 "+5V" H 6200 4340 50  0000 C CNN
 F 2 "" H 6200 4200 50  0001 C CNN
@@
 $EndComp
 $Comp
-L GND #PWR31
+L GND #PWR37
 U 1 1 5A026A49
 P 7700 5000
-F 0 "#PWR31" H 7700 4750 50  0001 C CNN
+F 0 "#PWR37" H 7700 4750 50  0001 C CNN
 F 1 "GND" H 7700 4850 50  0000 C CNN
 F 2 "" H 7700 5000 50  0001 C CNN
@@
 $EndComp
 $Comp
-L +5V #PWR34
+L +5V #PWR40
 U 1 1 5A027662
 P 8000 3750
-F 0 "#PWR34" H 8000 3600 50  0001 C CNN
+F 0 "#PWR40" H 8000 3600 50  0001 C CNN
 F 1 "+5V" H 8000 3890 50  0000 C CNN
 F 2 "" H 8000 3750 50  0001 C CNN
@@
 $EndComp
 $Comp
-L GND #PWR35
+L GND #PWR41
 U 1 1 5A02768A
 P 8000 4050
-F 0 "#PWR35" H 8000 3800 50  0001 C CNN
+F 0 "#PWR41" H 8000 3800 50  0001 C CNN
 F 1 "GND" H 8000 3900 50  0000 C CNN
 F 2 "" H 8000 4050 50  0001 C CNN
@@
 $EndComp
 $Comp
-L GND #PWR29
+L GND #PWR35
 U 1 1 5A027C7F
 P 6750 5150
-F 0 "#PWR29" H 6750 4900 50  0001 C CNN
+F 0 "#PWR35" H 6750 4900 50  0001 C CNN
 F 1 "GND" H 6750 5000 50  0000 C CNN
 F 2 "" H 6750 5150 50  0001 C CNN
@@
 $EndComp
 $Comp
-L +5V #PWR27
+L +5V #PWR33
 U 1 1 5A027DC0
 P 6550 5150
-F 0 "#PWR27" H 6550 5000 50  0001 C CNN
+F 0 "#PWR33" H 6550 5000 50  0001 C CNN
 F 1 "+5V" H 6550 5290 50  0000 C CNN
 F 2 "" H 6550 5150 50  0001 C CNN
@@
 Text HLabel 5400 4350 2    60   Input ~ 0
 START_INPUT
-Text Label 6950 1950 2    60   ~ 0
-CONTACT_REQ
 Text Notes 5450 4600 0    60   ~ 0
 GPIO
@@
 Text HLabel 7850 1850 2    60   Output ~ 0
 SEVCON_REV_12V_H
-Text HLabel 7850 1950 2    60   Output ~ 0
+Text HLabel 5400 3600 2    60   Output ~ 0
 CONTACT_REQ_12V_H
 Text HLabel 5250 1800 2    60   Output ~ 0
@@
 $EndComp
 $Comp
-L GND #PWR20
+L GND #PWR26
 U 1 1 5A042A3A
 P 3250 1500
-F 0 "#PWR20" H 3250 1250 50  0001 C CNN
+F 0 "#PWR26" H 3250 1250 50  0001 C CNN
 F 1 "GND" H 3250 1350 50  0000 C CNN
 F 2 "" H 3250 1500 50  0001 C CNN
@@
 $EndComp
 $Comp
-L +5V #PWR26
+L +5V #PWR32
 U 1 1 5A042E7E
 P 6550 2500
-F 0 "#PWR26" H 6550 2350 50  0001 C CNN
+F 0 "#PWR32" H 6550 2350 50  0001 C CNN
 F 1 "+5V" H 6550 2640 50  0000 C CNN
 F 2 "" H 6550 2500 50  0001 C CNN
@@
 $EndComp
 $Comp
-L GND #PWR28
+L GND #PWR34
 U 1 1 5A042EAC
 P 6700 3100
-F 0 "#PWR28" H 6700 2850 50  0001 C CNN
+F 0 "#PWR34" H 6700 2850 50  0001 C CNN
 F 1 "GND" H 6700 2950 50  0000 C CNN
 F 2 "" H 6700 3100 50  0001 C CNN
@@
 Connection ~ 3050 3400
 Wire Wire Line
-	3400 5500 3500 5500
-Wire Wire Line
-	3400 5500 3400 5850
+	3400 5600 3400 5850
 Wire Wire Line
 	3400 5600 3500 5600
 Wire Wire Line
 	3400 5700 3500 5700
-Connection ~ 3400 5600
 Connection ~ 3400 5700
 Wire Wire Line
@@
 	3350 3700 3500 3700
 Connection ~ 3350 3400
-Wire Wire Line
-	3350 3500 3500 3500
-Connection ~ 3350 3500
 Wire Wire Line
 	5400 4650 6700 4650
@@
 Text Label 6100 5100 0    60   ~ 0
 TX
+NoConn ~ 6950 2050
+NoConn ~ 7850 2050
+$Comp
+L ATMEGA328P-PU U?
+U 1 1 5A11510E
+P 4400 4500
+F 0 "U?" H 3650 5750 50  0000 L BNN
+F 1 "ATMEGA328P-PU" H 4800 3100 50  0000 L BNN
+F 2 "DIL28" H 4400 4500 50  0001 C CIN
+F 3 "" H 4400 4500 50  0001 C CNN
+	1    4400 4500
+	1    0    0    -1
+$EndComp
+NoConn ~ 6950 1950
+NoConn ~ 7850 1950
 $EndSCHEMATC

Commit message: added charger sd logic
Connections:
- net labels added: CONTACT_REQ_5V_H
- net labels removed: CONTACT_REQ_12V_H
Changed lines of the file:
@@
 SEVCON_REV_12V_H
 Text HLabel 5400 3600 2    60   Output ~ 0
-CONTACT_REQ_12V_H
+CONTACT_REQ_5V_H
 Text HLabel 5250 1800 2    60   Output ~ 0
 IMD_FLT_5V_L

Commit message: added most footprint associations
Parts:
- gave numbers to parts that had none: 1
- renumbered J1 to J6, J2 to J7, R4 to R6, R5 to R7, R6 to R8, U2 to U3, U4 to U5
Changed lines of the file:
@@
 $EndDescr
 $Comp
-L +5V #PWR24
+L +5V #PWR21
 U 1 1 5A023903
 P 3050 3300
-F 0 "#PWR24" H 3050 3150 50  0001 C CNN
+F 0 "#PWR21" H 3050 3150 50  0001 C CNN
 F 1 "+5V" H 3050 3440 50  0000 C CNN
 F 2 "" H 3050 3300 50  0001 C CNN
@@
 $EndComp
 $Comp
-L GND #PWR25
+L GND #PWR22
 U 1 1 5A0239BE
 P 3050 4150
-F 0 "#PWR25" H 3050 3900 50  0001 C CNN
+F 0 "#PWR22" H 3050 3900 50  0001 C CNN
 F 1 "GND" H 3050 4000 50  0000 C CNN
 F 2 "" H 3050 4150 50  0001 C CNN
@@
 $EndComp
 $Comp
-L GND #PWR27
+L GND #PWR24
 U 1 1 5A023B6E
 P 3400 5850
-F 0 "#PWR27" H 3400 5600 50  0001 C CNN
+F 0 "#PWR24" H 3400 5600 50  0001 C CNN
 F 1 "GND" H 3400 5700 50  0000 C CNN
 F 2 "" H 3400 5850 50  0001 C CNN
@@
 SCL
 $Comp
-L CD4050 U2
+L CD4050 U3
 U 1 1 5A0237EB
 P 4050 1600
-F 0 "U2" H 3900 1650 60  0000 C CNN
+F 0 "U3" H 3900 1650 60  0000 C CNN
 F 1 "CD4050" H 4000 1750 60  0000 C CNN
 F 2 "" H 4050 1600 60  0001 C CNN
@@
 TSMS_12V
 $Comp
-L GND #PWR29
+L GND #PWR26
 U 1 1 5A024854
 P 4750 1400
-F 0 "#PWR29" H 4750 1150 50  0001 C CNN
+F 0 "#PWR26" H 4750 1150 50  0001 C CNN
 F 1 "GND" H 4750 1250 50  0000 C CNN
 F 2 "" H 4750 1400 50  0001 C CNN
@@
 $EndComp
 $Comp
-L +12V #PWR28
+L +12V #PWR25
 U 1 1 5A024870
 P 3500 1050
-F 0 "#PWR28" H 3500 900 50  0001 C CNN
+F 0 "#PWR25" H 3500 900 50  0001 C CNN
 F 1 "+12V" H 3500 1190 50  0000 C CNN
 F 2 "" H 3500 1050 50  0001 C CNN
@@
 TSMS
 $Comp
-L CD40109 U4
+L CD40109 U5
 U 1 1 5A0250E7
 P 7400 1650
-F 0 "U4" H 7250 1700 60  0000 C CNN
+F 0 "U5" H 7250 1700 60  0000 C CNN
 F 1 "CD40109" H 7350 1800 60  0000 C CNN
 F 2 "" H 7400 1650 60  0001 C CNN
@@
 TSMS
 $Comp
-L +12V #PWR31
+L +12V #PWR28
 U 1 1 5A0259BE
 P 6350 2600
-F 0 "#PWR31" H 6350 2450 50  0001 C CNN
+F 0 "#PWR28" H 6350 2450 50  0001 C CNN
 F 1 "+12V" H 6350 2740 50  0000 C CNN
 F 2 "" H 6350 2600 50  0001 C CNN
@@
 $EndComp
 $Comp
-L +5V #PWR36
+L +5V #PWR33
 U 1 1 5A0259DC
 P 6800 2250
-F 0 "#PWR36" H 6800 2100 50  0001 C CNN
+F 0 "#PWR33" H 6800 2100 50  0001 C CNN
 F 1 "+5V" H 6800 2390 50  0000 C CNN
 F 2 "" H 6800 2250 50  0001 C CNN
@@
 $EndComp
 $Comp
-L GND #PWR39
+L GND #PWR36
 U 1 1 5A025A80
 P 8000 2650
-F 0 "#PWR39" H 8000 2400 50  0001 C CNN
+F 0 "#PWR36" H 8000 2400 50  0001 C CNN
 F 1 "GND" H 8000 2500 50  0000 C CNN
 F 2 "" H 8000 2650 50  0001 C CNN
@@
 $EndComp
 $Comp
-L +5V #PWR38
+L +5V #PWR35
 U 1 1 5A025B81
 P 8000 2250
-F 0 "#PWR38" H 8000 2100 50  0001 C CNN
+F 0 "#PWR35" H 8000 2100 50  0001 C CNN
 F 1 "+5V" H 8000 2390 50  0000 C CNN
 F 2 "" H 8000 2250 50  0001 C CNN
@@
 SEVCON_REV
 $Comp
-L R R4
+L R R6
 U 1 1 5A026097
 P 6200 4450
-F 0 "R4" V 6280 4450 50  0000 C CNN
+F 0 "R6" V 6280 4450 50  0000 C CNN
 F 1 "10k" V 6200 4450 50  0000 C CNN
 F 2 "" V 6130 4450 50  0001 C CNN
@@
 $EndComp
 $Comp
-L R R5
+L R R7
 U 1 1 5A026338
 P 6400 4450
-F 0 "R5" V 6480 4450 50  0000 C CNN
+F 0 "R7" V 6480 4450 50  0000 C CNN
 F 1 "10k" V 6400 4450 50  0000 C CNN
 F 2 "" V 6330 4450 50  0001 C CNN
@@
 $EndComp
 $Comp
-L +5V #PWR30
+L +5V #PWR27
 U 1 1 5A02647A
 P 6200 4200
-F 0 "#PWR30" H 6200 4050 50  0001 C CNN
+F 0 "#PWR27" H 6200 4050 50  0001 C CNN
 F 1 "+5V" H 6200 4340 50  0000 C CNN
 F 2 "" H 6200 4200 50  0001 C CNN
@@
 $EndComp
 $Comp
-L R R6
+L R R8
 U 1 1 5A026788
 P 6600 4450
-F 0 "R6" V 6680 4450 50  0000 C CNN
+F 0 "R8" V 6680 4450 50  0000 C CNN
 F 1 "10k" V 6600 4450 50  0000 C CNN
 F 2 "" V 6530 4450 50  0001 C CNN
@@
 $EndComp
 $Comp
-L GND #PWR37
+L GND #PWR34
 U 1 1 5A026A49
 P 7700 5000
-F 0 "#PWR37" H 7700 4750 50  0001 C CNN
+F 0 "#PWR34" H 7700 4750 50  0001 C CNN
 F 1 "GND" H 7700 4850 50  0000 C CNN
 F 2 "" H 7700 5000 50  0001 C CNN
@@
 $EndComp
 $Comp
-L Conn_02x03_Odd_Even J2
+L Conn_02x03_Odd_Even J7
 U 1 1 5A026A78
 P 7450 3900
-F 0 "J2" H 7500 4100 50  0000 C CNN
+F 0 "J7" H 7500 4100 50  0000 C CNN
 F 1 "ICSP" H 7500 3700 50  0000 C CNN
 F 2 "" H 7450 3900 50  0001 C CNN
@@
 $EndComp
 $Comp
-L +5V #PWR40
+L +5V #PWR37
 U 1 1 5A027662
 P 8000 3750
-F 0 "#PWR40" H 8000 3600 50  0001 C CNN
+F 0 "#PWR37" H 8000 3600 50  0001 C CNN
 F 1 "+5V" H 8000 3890 50  0000 C CNN
 F 2 "" H 8000 3750 50  0001 C CNN
@@
 $EndComp
 $Comp
-L GND #PWR41
+L GND #PWR38
 U 1 1 5A02768A
 P 8000 4050
-F 0 "#PWR41" H 8000 3800 50  0001 C CNN
+F 0 "#PWR38" H 8000 3800 50  0001 C CNN
 F 1 "GND" H 8000 3900 50  0000 C CNN
 F 2 "" H 8000 4050 50  0001 C CNN
@@
 $EndComp
 $Comp
-L Conn_01x06 J1
+L Conn_01x06 J6
 U 1 1 5A027A13
 P 7100 5350
-F 0 "J1" H 7100 5650 50  0000 C CNN
+F 0 "J6" H 7100 5650 50  0000 C CNN
 F 1 "FTDI" H 7100 4950 50  0000 C CNN
 F 2 "" H 7100 5350 50  0001 C CNN
@@
 $EndComp
 $Comp
-L GND #PWR35
+L GND #PWR32
 U 1 1 5A027C7F
 P 6750 5150
-F 0 "#PWR35" H 6750 4900 50  0001 C CNN
+F 0 "#PWR32" H 6750 4900 50  0001 C CNN
 F 1 "GND" H 6750 5000 50  0000 C CNN
 F 2 "" H 6750 5150 50  0001 C CNN
@@
 $EndComp
 $Comp
-L +5V #PWR33
+L +5V #PWR30
 U 1 1 5A027DC0
 P 6550 5150
-F 0 "#PWR33" H 6550 5000 50  0001 C CNN
+F 0 "#PWR30" H 6550 5000 50  0001 C CNN
 F 1 "+5V" H 6550 5290 50  0000 C CNN
 F 2 "" H 6550 5150 50  0001 C CNN
@@
 $EndComp
 $Comp
-L GND #PWR26
+L GND #PWR23
 U 1 1 5A042A3A
 P 3250 1500
-F 0 "#PWR26" H 3250 1250 50  0001 C CNN
+F 0 "#PWR23" H 3250 1250 50  0001 C CNN
 F 1 "GND" H 3250 1350 50  0000 C CNN
 F 2 "" H 3250 1500 50  0001 C CNN
@@
 $EndComp
 $Comp
-L +5V #PWR32
+L +5V #PWR29
 U 1 1 5A042E7E
 P 6550 2500
-F 0 "#PWR32" H 6550 2350 50  0001 C CNN
+F 0 "#PWR29" H 6550 2350 50  0001 C CNN
 F 1 "+5V" H 6550 2640 50  0000 C CNN
 F 2 "" H 6550 2500 50  0001 C CNN
@@
 $EndComp
 $Comp
-L GND #PWR34
+L GND #PWR31
 U 1 1 5A042EAC
 P 6700 3100
-F 0 "#PWR34" H 6700 2850 50  0001 C CNN
+F 0 "#PWR31" H 6700 2850 50  0001 C CNN
 F 1 "GND" H 6700 2950 50  0000 C CNN
 F 2 "" H 6700 3100 50  0001 C CNN
@@
 NoConn ~ 7850 2050
 $Comp
-L ATMEGA328P-PU U?
+L ATMEGA328P-PU U4
 U 1 1 5A11510E
 P 4400 4500
-F 0 "U?" H 3650 5750 50  0000 L BNN
+F 0 "U4" H 3650 5750 50  0000 L BNN
 F 1 "ATMEGA328P-PU" H 4800 3100 50  0000 L BNN
 F 2 "DIL28" H 4400 4500 50  0001 C CIN

Commit message: beginning board design
Parts:
- C1, C2, C3, C4, C5, C6: footprint (none) -> Capacitors_SMD:C_0805_HandSoldering
- J6: footprint (none) -> Pin_Headers:Pin_Header_Straight_1x06_Pitch2.54mm
- J7: footprint (none) -> Pin_Headers:Pin_Header_Straight_2x03_Pitch2.54mm
- R4: renamed from R6; footprint (none) -> Resistors_SMD:R_0805_HandSoldering
- R5: renamed from R7; footprint (none) -> Resistors_SMD:R_0805_HandSoldering
- R6: renamed from R8; footprint (none) -> Resistors_SMD:R_0805_HandSoldering
- SW1: renamed from SW2; footprint (none) -> Buttons_Switches_SMD:SW_SPST_PTS645
- U3: footprint (none) -> Housings_DIP:DIP-14_W8.89mm_SMDSocket_LongPads
- U4: footprint DIL28 -> Housings_DIP:DIP-28_W8.89mm_SMDSocket_LongPads
- U5: footprint (none) -> Housings_DIP:DIP-16_W8.89mm_SMDSocket_LongPads
Changed lines of the file:
@@
 $Descr A4 11693 8268
 encoding utf-8
-Sheet 3 4
+Sheet 2 4
 Title ""
 Date ""
@@
 $EndDescr
 $Comp
-L +5V #PWR21
+L +5V #PWR019
 U 1 1 5A023903
 P 3050 3300
-F 0 "#PWR21" H 3050 3150 50  0001 C CNN
+F 0 "#PWR019" H 3050 3150 50  0001 C CNN
 F 1 "+5V" H 3050 3440 50  0000 C CNN
 F 2 "" H 3050 3300 50  0001 C CNN
@@
 F 0 "C1" H 3075 3750 50  0000 L CNN
 F 1 "1u" H 3075 3550 50  0000 L CNN
-F 2 "" H 3088 3500 50  0001 C CNN
+F 2 "Capacitors_SMD:C_0805_HandSoldering" H 3088 3500 50  0001 C CNN
 F 3 "" H 3050 3650 50  0001 C CNN
 	1    3050 3650
@@
 $EndComp
 $Comp
-L GND #PWR22
+L GND #PWR020
 U 1 1 5A0239BE
 P 3050 4150
-F 0 "#PWR22" H 3050 3900 50  0001 C CNN
+F 0 "#PWR020" H 3050 3900 50  0001 C CNN
 F 1 "GND" H 3050 4000 50  0000 C CNN
 F 2 "" H 3050 4150 50  0001 C CNN
@@
 F 0 "C3" H 3275 4100 50  0000 L CNN
 F 1 ".1u" H 3275 3900 50  0000 L CNN
-F 2 "" H 3288 3850 50  0001 C CNN
+F 2 "Capacitors_SMD:C_0805_HandSoldering" H 3288 3850 50  0001 C CNN
 F 3 "" H 3250 4000 50  0001 C CNN
 	1    3250 4000
@@
 $EndComp
 $Comp
-L GND #PWR24
+L GND #PWR021
 U 1 1 5A023B6E
 P 3400 5850
-F 0 "#PWR24" H 3400 5600 50  0001 C CNN
+F 0 "#PWR021" H 3400 5600 50  0001 C CNN
 F 1 "GND" H 3400 5700 50  0000 C CNN
 F 2 "" H 3400 5850 50  0001 C CNN
@@
 F 0 "U3" H 3900 1650 60  0000 C CNN
 F 1 "CD4050" H 4000 1750 60  0000 C CNN
-F 2 "" H 4050 1600 60  0001 C CNN
+F 2 "Housings_DIP:DIP-14_W8.89mm_SMDSocket_LongPads" H 4050 1600 60  0001 C CNN
 F 3 "" H 4050 1600 60  0001 C CNN
 	1    4050 1600
@@
 TSMS_12V
 $Comp
-L GND #PWR26
+L GND #PWR022
 U 1 1 5A024854
 P 4750 1400
-F 0 "#PWR26" H 4750 1150 50  0001 C CNN
+F 0 "#PWR022" H 4750 1150 50  0001 C CNN
 F 1 "GND" H 4750 1250 50  0000 C CNN
 F 2 "" H 4750 1400 50  0001 C CNN
@@
 $EndComp
 $Comp
-L +12V #PWR25
+L +12V #PWR023
 U 1 1 5A024870
 P 3500 1050
-F 0 "#PWR25" H 3500 900 50  0001 C CNN
+F 0 "#PWR023" H 3500 900 50  0001 C CNN
 F 1 "+12V" H 3500 1190 50  0000 C CNN
 F 2 "" H 3500 1050 50  0001 C CNN
@@
 F 0 "U5" H 7250 1700 60  0000 C CNN
 F 1 "CD40109" H 7350 1800 60  0000 C CNN
-F 2 "" H 7400 1650 60  0001 C CNN
+F 2 "Housings_DIP:DIP-16_W8.89mm_SMDSocket_LongPads" H 7400 1650 60  0001 C CNN
 F 3 "" H 7400 1650 60  0001 C CNN
 	1    7400 1650
@@
 TSMS
 $Comp
-L +12V #PWR28
+L +12V #PWR024
 U 1 1 5A0259BE
 P 6350 2600
-F 0 "#PWR28" H 6350 2450 50  0001 C CNN
+F 0 "#PWR024" H 6350 2450 50  0001 C CNN
 F 1 "+12V" H 6350 2740 50  0000 C CNN
 F 2 "" H 6350 2600 50  0001 C CNN
@@
 $EndComp
 $Comp
-L +5V #PWR33
+L +5V #PWR025
 U 1 1 5A0259DC
 P 6800 2250
-F 0 "#PWR33" H 6800 2100 50  0001 C CNN
+F 0 "#PWR025" H 6800 2100 50  0001 C CNN
 F 1 "+5V" H 6800 2390 50  0000 C CNN
 F 2 "" H 6800 2250 50  0001 C CNN
@@
 $EndComp
 $Comp
-L GND #PWR36
+L GND #PWR026
 U 1 1 5A025A80
 P 8000 2650
-F 0 "#PWR36" H 8000 2400 50  0001 C CNN
+F 0 "#PWR026" H 8000 2400 50  0001 C CNN
 F 1 "GND" H 8000 2500 50  0000 C CNN
 F 2 "" H 8000 2650 50  0001 C CNN
@@
 $EndComp
 $Comp
-L +5V #PWR35
+L +5V #PWR027
 U 1 1 5A025B81
 P 8000 2250
-F 0 "#PWR35" H 8000 2100 50  0001 C CNN
+F 0 "#PWR027" H 8000 2100 50  0001 C CNN
 F 1 "+5V" H 8000 2390 50  0000 C CNN
 F 2 "" H 8000 2250 50  0001 C CNN
@@
 SEVCON_REV
 $Comp
-L R R6
+L R R4
 U 1 1 5A026097
 P 6200 4450
-F 0 "R6" V 6280 4450 50  0000 C CNN
+F 0 "R4" V 6280 4450 50  0000 C CNN
 F 1 "10k" V 6200 4450 50  0000 C CNN
-F 2 "" V 6130 4450 50  0001 C CNN
+F 2 "Resistors_SMD:R_0805_HandSoldering" V 6130 4450 50  0001 C CNN
 F 3 "" H 6200 4450 50  0001 C CNN
 	1    6200 4450
@@
 $EndComp
 $Comp
-L R R7
+L R R5
 U 1 1 5A026338
 P 6400 4450
-F 0 "R7" V 6480 4450 50  0000 C CNN
+F 0 "R5" V 6480 4450 50  0000 C CNN
 F 1 "10k" V 6400 4450 50  0000 C CNN
-F 2 "" V 6330 4450 50  0001 C CNN
+F 2 "Resistors_SMD:R_0805_HandSoldering" V 6330 4450 50  0001 C CNN
 F 3 "" H 6400 4450 50  0001 C CNN
 	1    6400 4450
@@
 $EndComp
 $Comp
-L +5V #PWR27
+L +5V #PWR028
 U 1 1 5A02647A
 P 6200 4200
-F 0 "#PWR27" H 6200 4050 50  0001 C CNN
+F 0 "#PWR028" H 6200 4050 50  0001 C CNN
 F 1 "+5V" H 6200 4340 50  0000 C CNN
 F 2 "" H 6200 4200 50  0001 C CNN
@@
 $EndComp
 $Comp
-L R R8
+L R R6
 U 1 1 5A026788
 P 6600 4450
-F 0 "R8" V 6680 4450 50  0000 C CNN
+F 0 "R6" V 6680 4450 50  0000 C CNN
 F 1 "10k" V 6600 4450 50  0000 C CNN
-F 2 "" V 6530 4450 50  0001 C CNN
+F 2 "Resistors_SMD:R_0805_HandSoldering" V 6530 4450 50  0001 C CNN
 F 3 "" H 6600 4450 50  0001 C CNN
 	1    6600 4450
@@
 $EndComp
 $Comp
-L SW_Push SW2
+L SW_Push SW1
 U 1 1 5A02695A
 P 7300 4850
-F 0 "SW2" H 7350 4950 50  0000 L CNN
+F 0 "SW1" H 7350 4950 50  0000 L CNN
 F 1 "SW_Push" H 7300 4790 50  0000 C CNN
-F 2 "" H 7300 5050 50  0001 C CNN
+F 2 "Buttons_Switches_SMD:SW_SPST_PTS645" H 7300 5050 50  0001 C CNN
 F 3 "" H 7300 5050 50  0001 C CNN
 	1    7300 4850
@@
 $EndComp
 $Comp
-L GND #PWR34
+L GND #PWR029
 U 1 1 5A026A49
 P 7700 5000
-F 0 "#PWR34" H 7700 4750 50  0001 C CNN
+F 0 "#PWR029" H 7700 4750 50  0001 C CNN
 F 1 "GND" H 7700 4850 50  0000 C CNN
 F 2 "" H 7700 5000 50  0001 C CNN
@@
 F 0 "J7" H 7500 4100 50  0000 C CNN
 F 1 "ICSP" H 7500 3700 50  0000 C CNN
-F 2 "" H 7450 3900 50  0001 C CNN
+F 2 "Pin_Headers:Pin_Header_Straight_2x03_Pitch2.54mm" H 7450 3900 50  0001 C CNN
 F 3 "" H 7450 3900 50  0001 C CNN
 	1    7450 3900
@@
 $EndComp
 $Comp
-L +5V #PWR37
+L +5V #PWR030
 U 1 1 5A027662
 P 8000 3750
-F 0 "#PWR37" H 8000 3600 50  0001 C CNN
+F 0 "#PWR030" H 8000 3600 50  0001 C CNN
 F 1 "+5V" H 8000 3890 50  0000 C CNN
 F 2 "" H 8000 3750 50  0001 C CNN
@@
 $EndComp
 $Comp
-L GND #PWR38
+L GND #PWR031
 U 1 1 5A02768A
 P 8000 4050
-F 0 "#PWR38" H 8000 3800 50  0001 C CNN
+F 0 "#PWR031" H 8000 3800 50  0001 C CNN
 F 1 "GND" H 8000 3900 50  0000 C CNN
 F 2 "" H 8000 4050 50  0001 C CNN
@@
 F 0 "J6" H 7100 5650 50  0000 C CNN
 F 1 "FTDI" H 7100 4950 50  0000 C CNN
-F 2 "" H 7100 5350 50  0001 C CNN
+F 2 "Pin_Headers:Pin_Header_Straight_1x06_Pitch2.54mm" H 7100 5350 50  0001 C CNN
 F 3 "" H 7100 5350 50  0001 C CNN
 	1    7100 5350
@@
 $EndComp
 $Comp
-L GND #PWR32
+L GND #PWR032
 U 1 1 5A027C7F
 P 6750 5150
-F 0 "#PWR32" H 6750 4900 50  0001 C CNN
+F 0 "#PWR032" H 6750 4900 50  0001 C CNN
 F 1 "GND" H 6750 5000 50  0000 C CNN
 F 2 "" H 6750 5150 50  0001 C CNN
@@
 $EndComp
 $Comp
-L +5V #PWR30
+L +5V #PWR033
 U 1 1 5A027DC0
 P 6550 5150
-F 0 "#PWR30" H 6550 5000 50  0001 C CNN
+F 0 "#PWR033" H 6550 5000 50  0001 C CNN
 F 1 "+5V" H 6550 5290 50  0000 C CNN
 F 2 "" H 6550 5150 50  0001 C CNN
@@
 F 0 "C5" H 6675 5750 50  0000 L CNN
 F 1 "1u" H 6675 5550 50  0000 L CNN
-F 2 "" H 6688 5500 50  0001 C CNN
+F 2 "Capacitors_SMD:C_0805_HandSoldering" H 6688 5500 50  0001 C CNN
 F 3 "" H 6650 5650 50  0001 C CNN
 	1    6650 5650
@@
 F 0 "C2" H 3275 1400 50  0000 L CNN
 F 1 "1u" H 3275 1200 50  0000 L CNN
-F 2 "" H 3288 1150 50  0001 C CNN
+F 2 "Capacitors_SMD:C_0805_HandSoldering" H 3288 1150 50  0001 C CNN
 F 3 "" H 3250 1300 50  0001 C CNN
 	1    3250 1300
@@
 $EndComp
 $Comp
-L GND #PWR23
+L GND #PWR034
 U 1 1 5A042A3A
 P 3250 1500
-F 0 "#PWR23" H 3250 1250 50  0001 C CNN
+F 0 "#PWR034" H 3250 1250 50  0001 C CNN
 F 1 "GND" H 3250 1350 50  0000 C CNN
 F 2 "" H 3250 1500 50  0001 C CNN
@@
 $EndComp
 $Comp
-L +5V #PWR29
+L +5V #PWR035
 U 1 1 5A042E7E
 P 6550 2500
-F 0 "#PWR29" H 6550 2350 50  0001 C CNN
+F 0 "#PWR035" H 6550 2350 50  0001 C CNN
 F 1 "+5V" H 6550 2640 50  0000 C CNN
 F 2 "" H 6550 2500 50  0001 C CNN
@@
 $EndComp
 $Comp
-L GND #PWR31
+L GND #PWR036
 U 1 1 5A042EAC
 P 6700 3100
-F 0 "#PWR31" H 6700 2850 50  0001 C CNN
+F 0 "#PWR036" H 6700 2850 50  0001 C CNN
 F 1 "GND" H 6700 2950 50  0000 C CNN
 F 2 "" H 6700 3100 50  0001 C CNN
@@
 F 0 "C6" H 6825 2950 50  0000 L CNN
 F 1 "1u" H 6825 2750 50  0000 L CNN
-F 2 "" H 6838 2700 50  0001 C CNN
+F 2 "Capacitors_SMD:C_0805_HandSoldering" H 6838 2700 50  0001 C CNN
 F 3 "" H 6800 2850 50  0001 C CNN
 	1    6800 2850
@@
 F 0 "C4" H 6625 2950 50  0000 L CNN
 F 1 "1u" H 6625 2750 50  0000 L CNN
-F 2 "" H 6638 2700 50  0001 C CNN
+F 2 "Capacitors_SMD:C_0805_HandSoldering" H 6638 2700 50  0001 C CNN
 F 3 "" H 6600 2850 50  0001 C CNN
 	1    6600 2850
@@
 F 0 "U4" H 3650 5750 50  0000 L BNN
 F 1 "ATMEGA328P-PU" H 4800 3100 50  0000 L BNN
-F 2 "DIL28" H 4400 4500 50  0001 C CIN
+F 2 "Housings_DIP:DIP-28_W8.89mm_SMDSocket_LongPads" H 4400 4500 50  0001 C CIN
 F 3 "" H 4400 4500 50  0001 C CNN
 	1    4400 4500
