File: Logic.sch (KiCad schematic (older format))
At the start: 15 parts, among them J6 FTDI, J7 ICSP, SW1 SW_Push, U3 CD4050, U4 ATMEGA328P-PU, U5 CD40109

Commit message: beginning floorplan
Connections:
- net labels added: RST
Changed lines of the file:
@@
 $EndDescr
 $Comp
-L +5V #PWR019
+L +5V #PWR022
 U 1 1 5A023903
 P 3050 3300
-F 0 "#PWR019" H 3050 3150 50  0001 C CNN
+F 0 "#PWR022" H 3050 3150 50  0001 C CNN
 F 1 "+5V" H 3050 3440 50  0000 C CNN
 F 2 "" H 3050 3300 50  0001 C CNN
@@
 $EndComp
 $Comp
-L GND #PWR020
+L GND #PWR023
 U 1 1 5A0239BE
 P 3050 4150
-F 0 "#PWR020" H 3050 3900 50  0001 C CNN
+F 0 "#PWR023" H 3050 3900 50  0001 C CNN
 F 1 "GND" H 3050 4000 50  0000 C CNN
 F 2 "" H 3050 4150 50  0001 C CNN
@@
 $EndComp
 $Comp
-L GND #PWR021
+L GND #PWR024
 U 1 1 5A023B6E
 P 3400 5850
-F 0 "#PWR021" H 3400 5600 50  0001 C CNN
+F 0 "#PWR024" H 3400 5600 50  0001 C CNN
 F 1 "GND" H 3400 5700 50  0000 C CNN
 F 2 "" H 3400 5850 50  0001 C CNN
@@
 TSMS_12V
 $Comp
-L GND #PWR022
+L GND #PWR025
 U 1 1 5A024854
 P 4750 1400
-F 0 "#PWR022" H 4750 1150 50  0001 C CNN
+F 0 "#PWR025" H 4750 1150 50  0001 C CNN
 F 1 "GND" H 4750 1250 50  0000 C CNN
 F 2 "" H 4750 1400 50  0001 C CNN
@@
 $EndComp
 $Comp
-L +12V #PWR023
+L +12V #PWR026
 U 1 1 5A024870
 P 3500 1050
-F 0 "#PWR023" H 3500 900 50  0001 C CNN
+F 0 "#PWR026" H 3500 900 50  0001 C CNN
 F 1 "+12V" H 3500 1190 50  0000 C CNN
 F 2 "" H 3500 1050 50  0001 C CNN
@@
 TSMS
 $Comp
-L +12V #PWR024
+L +12V #PWR027
 U 1 1 5A0259BE
 P 6350 2600
-F 0 "#PWR024" H 6350 2450 50  0001 C CNN
+F 0 "#PWR027" H 6350 2450 50  0001 C CNN
 F 1 "+12V" H 6350 2740 50  0000 C CNN
 F 2 "" H 6350 2600 50  0001 C CNN
@@
 $EndComp
 $Comp
-L +5V #PWR025
+L +5V #PWR028
 U 1 1 5A0259DC
 P 6800 2250
-F 0 "#PWR025" H 6800 2100 50  0001 C CNN
+F 0 "#PWR028" H 6800 2100 50  0001 C CNN
 F 1 "+5V" H 6800 2390 50  0000 C CNN
 F 2 "" H 6800 2250 50  0001 C CNN
@@
 $EndComp
 $Comp
-L GND #PWR026
+L GND #PWR029
 U 1 1 5A025A80
 P 8000 2650
-F 0 "#PWR026" H 8000 2400 50  0001 C CNN
+F 0 "#PWR029" H 8000 2400 50  0001 C CNN
 F 1 "GND" H 8000 2500 50  0000 C CNN
 F 2 "" H 8000 2650 50  0001 C CNN
@@
 $EndComp
 $Comp
-L +5V #PWR027
+L +5V #PWR030
 U 1 1 5A025B81
 P 8000 2250
-F 0 "#PWR027" H 8000 2100 50  0001 C CNN
+F 0 "#PWR030" H 8000 2100 50  0001 C CNN
 F 1 "+5V" H 8000 2390 50  0000 C CNN
 F 2 "" H 8000 2250 50  0001 C CNN
@@
 $EndComp
 $Comp
-L +5V #PWR028
+L +5V #PWR031
 U 1 1 5A02647A
 P 6200 4200
-F 0 "#PWR028" H 6200 4050 50  0001 C CNN
+F 0 "#PWR031" H 6200 4050 50  0001 C CNN
 F 1 "+5V" H 6200 4340 50  0000 C CNN
 F 2 "" H 6200 4200 50  0001 C CNN
@@
 $EndComp
 $Comp
-L GND #PWR029
+L GND #PWR032
 U 1 1 5A026A49
 P 7700 5000
-F 0 "#PWR029" H 7700 4750 50  0001 C CNN
+F 0 "#PWR032" H 7700 4750 50  0001 C CNN
 F 1 "GND" H 7700 4850 50  0000 C CNN
 F 2 "" H 7700 5000 50  0001 C CNN
@@
 $EndComp
 $Comp
-L +5V #PWR030
+L +5V #PWR033
 U 1 1 5A027662
 P 8000 3750
-F 0 "#PWR030" H 8000 3600 50  0001 C CNN
+F 0 "#PWR033" H 8000 3600 50  0001 C CNN
 F 1 "+5V" H 8000 3890 50  0000 C CNN
 F 2 "" H 8000 3750 50  0001 C CNN
@@
 $EndComp
 $Comp
-L GND #PWR031
+L GND #PWR034
 U 1 1 5A02768A
 P 8000 4050
-F 0 "#PWR031" H 8000 3800 50  0001 C CNN
+F 0 "#PWR034" H 8000 3800 50  0001 C CNN
 F 1 "GND" H 8000 3900 50  0000 C CNN
 F 2 "" H 8000 4050 50  0001 C CNN
@@
 $EndComp
 $Comp
-L GND #PWR032
+L GND #PWR035
 U 1 1 5A027C7F
 P 6750 5150
-F 0 "#PWR032" H 6750 4900 50  0001 C CNN
+F 0 "#PWR035" H 6750 4900 50  0001 C CNN
 F 1 "GND" H 6750 5000 50  0000 C CNN
 F 2 "" H 6750 5150 50  0001 C CNN
@@
 $EndComp
 $Comp
-L +5V #PWR033
+L +5V #PWR036
 U 1 1 5A027DC0
 P 6550 5150
-F 0 "#PWR033" H 6550 5000 50  0001 C CNN
+F 0 "#PWR036" H 6550 5000 50  0001 C CNN
 F 1 "+5V" H 6550 5290 50  0000 C CNN
 F 2 "" H 6550 5150 50  0001 C CNN
@@
 $EndComp
 $Comp
-L GND #PWR034
+L GND #PWR037
 U 1 1 5A042A3A
 P 3250 1500
-F 0 "#PWR034" H 3250 1250 50  0001 C CNN
+F 0 "#PWR037" H 3250 1250 50  0001 C CNN
 F 1 "GND" H 3250 1350 50  0000 C CNN
 F 2 "" H 3250 1500 50  0001 C CNN
@@
 $EndComp
 $Comp
-L +5V #PWR035
+L +5V #PWR038
 U 1 1 5A042E7E
 P 6550 2500
-F 0 "#PWR035" H 6550 2350 50  0001 C CNN
+F 0 "#PWR038" H 6550 2350 50  0001 C CNN
 F 1 "+5V" H 6550 2640 50  0000 C CNN
 F 2 "" H 6550 2500 50  0001 C CNN
@@
 $EndComp
 $Comp
-L GND #PWR036
+L GND #PWR039
 U 1 1 5A042EAC
 P 6700 3100
-F 0 "#PWR036" H 6700 2850 50  0001 C CNN
+F 0 "#PWR039" H 6700 2850 50  0001 C CNN
 F 1 "GND" H 6700 2950 50  0000 C CNN
 F 2 "" H 6700 3100 50  0001 C CNN
@@
 	3500 1700 3600 1700
 Wire Wire Line
-	6350 2650 6950 2650
-Wire Wire Line
 	7850 2650 8000 2650
 Wire Wire Line
@@
 Connection ~ 6900 2250
 Wire Wire Line
-	6550 2550 6950 2550
-Wire Wire Line
 	6200 4600 6200 4650
 Connection ~ 6200 4650
@@
 	6350 2650 6350 2600
 Wire Wire Line
-	6600 2700 6600 2650
-Connection ~ 6600 2650
-Wire Wire Line
 	6800 2700 6800 2550
-Connection ~ 6800 2550
 Wire Wire Line
 	6600 3000 6600 3050
@@
 NoConn ~ 6950 1950
 NoConn ~ 7850 1950
+Text Label 6100 4850 0    60   ~ 0
+RST
+Wire Wire Line
+	6550 2550 6950 2550
+Connection ~ 6800 2550
+Wire Wire Line
+	6350 2650 6950 2650
+Wire Wire Line
+	6600 2650 6600 2700
+Connection ~ 6600 2650
 $EndSCHEMATC

Commit message: winter break changes
Parts:
- C1, C2, C3, C4, C5, C6: footprint Capacitors_SMD:C_0805_HandSoldering -> Capacitors_SMD:C_0603_HandSoldering
- R4, R5, R6: footprint Resistors_SMD:R_0805_HandSoldering -> Resistors_SMD:R_0603_HandSoldering
Changed lines of the file:
@@
 F 0 "C1" H 3075 3750 50  0000 L CNN
 F 1 "1u" H 3075 3550 50  0000 L CNN
-F 2 "Capacitors_SMD:C_0805_HandSoldering" H 3088 3500 50  0001 C CNN
+F 2 "Capacitors_SMD:C_0603_HandSoldering" H 3088 3500 50  0001 C CNN
 F 3 "" H 3050 3650 50  0001 C CNN
 	1    3050 3650
@@
 F 0 "C3" H 3275 4100 50  0000 L CNN
 F 1 ".1u" H 3275 3900 50  0000 L CNN
-F 2 "Capacitors_SMD:C_0805_HandSoldering" H 3288 3850 50  0001 C CNN
+F 2 "Capacitors_SMD:C_0603_HandSoldering" H 3288 3850 50  0001 C CNN
 F 3 "" H 3250 4000 50  0001 C CNN
 	1    3250 4000
@@
 F 0 "R4" V 6280 4450 50  0000 C CNN
 F 1 "10k" V 6200 4450 50  0000 C CNN
-F 2 "Resistors_SMD:R_0805_HandSoldering" V 6130 4450 50  0001 C CNN
+F 2 "Resistors_SMD:R_0603_HandSoldering" V 6130 4450 50  0001 C CNN
 F 3 "" H 6200 4450 50  0001 C CNN
 	1    6200 4450
@@
 F 0 "R5" V 6480 4450 50  0000 C CNN
 F 1 "10k" V 6400 4450 50  0000 C CNN
-F 2 "Resistors_SMD:R_0805_HandSoldering" V 6330 4450 50  0001 C CNN
+F 2 "Resistors_SMD:R_0603_HandSoldering" V 6330 4450 50  0001 C CNN
 F 3 "" H 6400 4450 50  0001 C CNN
 	1    6400 4450
@@
 F 0 "R6" V 6680 4450 50  0000 C CNN
 F 1 "10k" V 6600 4450 50  0000 C CNN
-F 2 "Resistors_SMD:R_0805_HandSoldering" V 6530 4450 50  0001 C CNN
+F 2 "Resistors_SMD:R_0603_HandSoldering" V 6530 4450 50  0001 C CNN
 F 3 "" H 6600 4450 50  0001 C CNN
 	1    6600 4450
@@
 F 0 "C5" H 6675 5750 50  0000 L CNN
 F 1 "1u" H 6675 5550 50  0000 L CNN
-F 2 "Capacitors_SMD:C_0805_HandSoldering" H 6688 5500 50  0001 C CNN
+F 2 "Capacitors_SMD:C_0603_HandSoldering" H 6688 5500 50  0001 C CNN
 F 3 "" H 6650 5650 50  0001 C CNN
 	1    6650 5650
@@
 F 0 "C2" H 3275 1400 50  0000 L CNN
 F 1 "1u" H 3275 1200 50  0000 L CNN
-F 2 "Capacitors_SMD:C_0805_HandSoldering" H 3288 1150 50  0001 C CNN
+F 2 "Capacitors_SMD:C_0603_HandSoldering" H 3288 1150 50  0001 C CNN
 F 3 "" H 3250 1300 50  0001 C CNN
 	1    3250 1300
@@
 F 0 "C6" H 6825 2950 50  0000 L CNN
 F 1 "1u" H 6825 2750 50  0000 L CNN
-F 2 "Capacitors_SMD:C_0805_HandSoldering" H 6838 2700 50  0001 C CNN
+F 2 "Capacitors_SMD:C_0603_HandSoldering" H 6838 2700 50  0001 C CNN
 F 3 "" H 6800 2850 50  0001 C CNN
 	1    6800 2850
@@
 F 0 "C4" H 6625 2950 50  0000 L CNN
 F 1 "1u" H 6625 2750 50  0000 L CNN
-F 2 "Capacitors_SMD:C_0805_HandSoldering" H 6638 2700 50  0001 C CNN
+F 2 "Capacitors_SMD:C_0603_HandSoldering" H 6638 2700 50  0001 C CNN
 F 3 "" H 6600 2850 50  0001 C CNN
 	1    6600 2850

Commit message: finished routing
Parts:
- added C15, C16, C17: C, Capacitors_SMD:C_0805_HandSoldering, symbol C
- added Y1: Crystal, Crystals:Crystal_SMD_HC49-SD_HandSoldering, symbol Crystal
- C1, C2, C3, C4, C5, C6: footprint Capacitors_SMD:C_0603_HandSoldering -> Resistors_SMD:R_0805_HandSoldering
- R4, R5, R6: footprint Resistors_SMD:R_0603_HandSoldering -> Resistors_SMD:R_0805_HandSoldering
- U3: footprint Housings_DIP:DIP-14_W8.89mm_SMDSocket_LongPads -> Housings_DIP:DIP-16_W8.89mm_SMDSocket_LongPads
Connections:
- wire segments 80 -> 93
- no-connect marks 6 -> 4
Other:
- note removed: "Crystal"
- moved on the sheet: C1, C3, J7, SW1

Commit message: final design competition 2018
Parts:
- C17: value C -> 1u
Connections:
- net labels removed: SECON_FWD
Changed lines of the file:
@@
 $EndComp
 Text Label 4250 3400 0    60   ~ 0
-SECON_FWD
+SEVCON_FWD
 Text Label 4250 3500 0    60   ~ 0
 SEVCON_REV
@@
 P 7300 5100
 F 0 "C17" H 7325 5200 50  0000 L CNN
-F 1 "C" H 7325 5000 50  0000 L CNN
+F 1 "1u" H 7325 5000 50  0000 L CNN
 F 2 "Capacitors_SMD:C_0805_HandSoldering" H 7338 4950 50  0001 C CNN
 F 3 "" H 7300 5100 50  0001 C CNN
