File: Motherboard.kicad_pcb (KiCad board)
At the start: 2 copper layers, 44 parts, among them J3 Conn_01x14_Male, J4 Conn_01x14_Male, J5 Conn_01x14_Male, J6 FTDI, J7 ICSP, K1 IMD_RELAY, K2 IMD_LATCH, K3 BMS_RELAY, SW1 SW_Push, U1 LM7805_TO220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

Commit message: working on bms connectors
Other:
- net class Signal added: clearance 0.2, trace_width 0.5, via_dia 0.5, via_drill 0.4
Changed lines of the file:
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@@
 (kicad_pcb (version 4) (host pcbnew 4.0.7-e2-6376~58~ubuntu16.04.1)
   (general
-    (links 0)
-    (no_connects 132)
+    (links 143)
+    (no_connects 138)
     (area 0 0 0 0)
     (thickness 1.6)
@@
     (add_net VCC)
   )
+  (net_class Signal ""
+    (clearance 0.2)
+    (trace_width 0.5)
+    (via_dia 0.5)
+    (via_drill 0.4)
+    (uvia_dia 0.3)
+    (uvia_drill 0.1)
+  )
   (module Capacitors_SMD:C_0805_HandSoldering (layer F.Cu)

Commit message: beginning floorplan
Parts:
- moved U1 190.7 mm to (194.3, 94.6)
- moved F1 171.7 mm to (190.5, 88.3), turned to 90 degrees
- moved F11 165.2 mm to (210.8, 88.3), turned to 90 degrees
- moved F10 155.9 mm to (200.7, 88.3), turned to 90 degrees
- moved J6 132.4 mm to (160.8, 95.3)
- moved J7 132.2 mm to (179.7, 87.0), turned to 270 degrees
- moved R1 104.6 mm to (182.5, 107.2)
- moved U4 104.6 mm to (172.3, 116.1)
- moved SW1 102.5 mm to (152.7, 96.4), turned to 270 degrees
- moved U5 101.8 mm to (127.6, 125.7)
- moved F9 97.3 mm to (104.6, 137.1), turned to 180 degrees
- moved U6 94.8 mm to (148.0, 126.4)
- moved J5 94.4 mm to (59.7, 151.1)
- moved F2 92.9 mm to (108.0, 93.3), turned to 180 degrees
- moved D3 86.0 mm to (59.7, 110.5)
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Connections:
- net Net-(C5-Pad2) renamed /Logic/RST
- F1 pad 1: +5V -> Net-(F1-Pad1)
- F1 pad 2: Net-(F1-Pad2) -> +12V
- F3 pad 1: Net-(F3-Pad1) -> /RTDS+
- F4 pad 1: Net-(F4-Pad1) -> /BATT_FAN+
- F5 pad 1: Net-(F5-Pad1) -> /BRK_LIGHT+
- F6 pad 1: Net-(F6-Pad1) -> /RAD_FAN+
- F7 pad 1: Net-(F7-Pad1) -> /PUMP+
- F8 pad 1: Net-(F8-Pad1) -> /LAP_TIMER+
- J4 pad 10: /IMD_FLT -> Net-(F12-Pad1)
- J4 pad 11: GND -> /IMD_RST+
- J4 pad 12: /IMD_RST+ -> /IMD_RST-
- J4 pad 13: /IMD_RST- -> GND
- J4 pad 4: Net-(F9-Pad1) -> GND
- J4 pad 5: /SEVCON_FWD -> /SEVCON_FLT
- J4 pad 6: /SEVCON_REV -> Net-(F9-Pad1)
- J4 pad 7: /SEVCON_FLT -> /SEVCON_FWD
- J4 pad 8: GND -> /SEVCON_REV
- J4 pad 9: Net-(F12-Pad1) -> /IMD_FLT
- J5 pad 1: Net-(F3-Pad1) -> /BATT_FAN+
- J5 pad 10: +12V -> /TSMS
- J5 pad 11: /SD_CKT- -> /BOTS
- J5 pad 12: /TSMS -> Net-(J5-Pad12)
- J5 pad 13: /BOTS -> +12V
- J5 pad 14: Net-(J5-Pad14) -> /SD_CKT-
- J5 pad 2: /RTDS- -> /BATT_FAN-
- J5 pad 3: Net-(F4-Pad1) -> /RAD_FAN+
- J5 pad 4: /FAN- -> /PUMP+
- J5 pad 5: Net-(F5-Pad1) -> /LAP_TIMER+
- J5 pad 6: /BRK_SW -> /RTDS+
- J5 pad 7: Net-(F6-Pad1) -> /RTDS-
- J5 pad 8: Net-(F7-Pad1) -> /BRK_LIGHT+
- J5 pad 9: Net-(F8-Pad1) -> /BRK_SW
- U1 pad 1: +12V -> Net-(F1-Pad1)
- U1 pad 3: Net-(F1-Pad2) -> +5V
- U2 pad 14: VCC -> +5V
- U5 pad 1: (no net) -> +5V
- U5 pad 12: +5V -> Net-(U5-Pad12)
- U5 pad 15: Net-(U5-Pad15) -> +5V
- U5 pad 16: GND -> +12V
- U5 pad 7: (no net) -> +5V
- U5 pad 8: (no net) -> GND
- U5 pad 9: (no net) -> +5V
- U6 pad 14: VCC -> +5V
Routing:
- net /IMD_FLT_12V_LED_H: track 0.00 -> 108.3 mm
- net Net-(J7-Pad3): track 0.00 -> 57.0 mm
- net Net-(J7-Pad1): track 0.00 -> 55.5 mm
- net /BATT_FAN+: track 0.00 -> 50.5 mm
- net /BRK_LIGHT+: track 0.00 -> 50.3 mm
- net (no net): track 0.00 -> 47.6 mm, vias 0 -> 1
- net /LAP_TIMER+: track 0.00 -> 46.1 mm
- net /SCL: track 0.00 -> 43.2 mm
- net Net-(F12-Pad1): track 0.00 -> 42.3 mm
- net /SDA: track 0.00 -> 40.0 mm
- net /RTDS+: track 0.00 -> 39.5 mm
- net /Logic/RTDS: track 0.00 -> 33.8 mm
- net +12V: track 29.3 -> 62.8 mm
- net /SD_CKT-: track 0.00 -> 32.8 mm
- net /ShutdownCircuit/IMD_RST-: track 30.4 -> 0.00 mm
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- added copper zone on F.Cu, net +12V
- added copper zone on F.Cu, net +5V
- added copper zone on B.Cu, net GND
Other:
- board text added: "BMS Bullshit"

Commit message: winter break changes
Parts:
- added C7: CP, Capacitors_THT:CP_Radial_D8.0mm_P5.00mm, F.Cu at (142.9, 145.4)
- added C8: CP, Capacitors_THT:CP_Radial_D8.0mm_P5.00mm, F.Cu at (151.8, 145.4)
- added J1: Conn_01x16_Male, Connectors_Molex:Molex_MiniFit-JR-5556-16A_2x08x4.20mm_Straight, F.Cu at (106.0, 87.0)
- added J2: Conn_01x04_Male, Connectors_Molex:Molex_MiniFit-JR-5556-04A_2x02x4.20mm_Straight, F.Cu at (114.3, 129.5)
- added J8: Conn_01x06_Male, Connectors_Molex:Molex_MiniFit-JR-5556-06A_2x03x4.20mm_Straight, F.Cu at (61.0, 81.9)
- added Q1: Q_NMOS_DGS, TO_SOT_Packages_SMD:TO-263-2, F.Cu at (22.9, 94.0)
- added Q2: Q_NMOS_DGS, TO_SOT_Packages_SMD:TO-263-2, F.Cu at (35.6, 94.0)
- added Q3: Q_NMOS_DGS, TO_SOT_Packages_SMD:TO-263-2, F.Cu at (81.3, 139.7)
- added Q4: Q_NMOS_DGS, TO_SOT_Packages_SMD:TO-263-2, F.Cu at (63.5, 139.7)
- added R10: R, Resistors_SMD:R_0603_HandSoldering, F.Cu at (69.8, 102.2)
- added R7: R, Resistors_SMD:R_0603_HandSoldering, F.Cu at (142.2, 151.1)
- added R8: R, Resistors_SMD:R_0603_HandSoldering, F.Cu at (151.1, 151.1)
- added R9: R, Resistors_SMD:R_0603_HandSoldering, F.Cu at (87.6, 102.2)
- C1, C2, C3, C4, C5, C6: footprint Capacitors_SMD:C_0805_HandSoldering -> Capacitors_SMD:C_0603_HandSoldering
- D1, D3: footprint LEDs:LED_0805_HandSoldering -> LEDs:LED_0603_HandSoldering
- R1, R2, R4, R5, R6: footprint Resistors_SMD:R_0805_HandSoldering -> Resistors_SMD:R_0603_HandSoldering
- moved K2 28.2 mm to (99.1, 104.1)
- moved F13 23.5 mm to (45.7, 99.1), turned to 90 degrees
- moved J5 16.6 mm to (43.2, 152.4)
- moved D4 15.9 mm to (63.5, 97.2)
- moved D2 15.6 mm to (81.3, 96.5)
- moved U5 9.44 mm to (136.5, 128.9)
- moved D3 9.09 mm to (63.5, 102.2), turned to 180 degrees
- moved D1 8.28 mm to (81.3, 102.2), turned to 180 degrees
- moved C6 8.26 mm to (132.1, 116.8)
- moved K1 7.73 mm to (81.3, 109.2)
- moved K3 7.73 mm to (63.5, 109.2)
- moved F1 5.99 mm to (185.4, 91.4)
- moved F10 5.99 mm to (195.6, 91.4)
- moved F11 5.99 mm to (205.7, 91.4)
- moved C1 5.83 mm to (165.1, 121.9)
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Connections:
- D1 pad 2: /ShutdownCircuit/IMD_RST- -> /IMD_RST-
- D2 pad 1: /ShutdownCircuit/IMD_RST- -> /IMD_RST-
- J4 pad 11: /IMD_RST+ -> +12V
- K1 pad 1: /ShutdownCircuit/IMD_RST- -> /IMD_RST-
- K2 pad 1: /ShutdownCircuit/IMD_RST- -> /IMD_RST-
- K2 pad 3: /ShutdownCircuit/IMD_RST- -> /IMD_RST-
Routing:
- net /IMD_RST-: track 0.00 -> 110.5 mm, vias 0 -> 1
- net /IMD_FLT_12V_LED_H: track 108.3 -> 0.00 mm
- net Net-(D2-Pad2): track 0.00 -> 77.9 mm
- net Net-(D4-Pad2): track 0.00 -> 59.2 mm
- net /RTDS-: track 0.00 -> 54.1 mm
- net Net-(J7-Pad4): track 9.32 -> 54.7 mm, vias 1 -> 2
- net /RTDS+: track 39.5 -> 0.00 mm
- net /SCL: track 43.2 -> 3.98 mm
- net /SDA: track 40.0 -> 3.98 mm
- net /Logic/RTDS: track 33.8 -> 0.00 mm
- net /BOTS: track 0.00 -> 30.4 mm
- net /START_INPUT: track 30.3 -> 0.00 mm
- net (no net): track 47.6 -> 74.6 mm, vias 1 -> 3
- net +12V: track 62.8 -> 38.1 mm
- net /BRK_LIGHT+: track 50.3 -> 28.2 mm
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
Commit message: finished routing
Parts:
- added C10: C, Resistors_SMD:R_0805_HandSoldering, F.Cu at (109.5, 36.1)
- added C11: C, Resistors_SMD:R_0805_HandSoldering, F.Cu at (114.6, 34.0)
- added C12: C, Resistors_SMD:R_0805_HandSoldering, F.Cu at (114.6, 36.1)
- added C13: C, Capacitors_SMD:C_0805_HandSoldering, F.Cu at (141.7, 38.0)
- added C14: C, Capacitors_SMD:C_0805_HandSoldering, F.Cu at (145.4, 38.1)
- added C15: C, Capacitors_SMD:C_0805_HandSoldering, F.Cu at (156.8, 52.1)
- added C16: C, Capacitors_SMD:C_0805_HandSoldering, F.Cu at (156.8, 64.8)
- added C17: C, Capacitors_SMD:C_0805_HandSoldering, F.Cu at (160.1, 31.9)
- added C18: C, Resistors_SMD:R_0805_HandSoldering, F.Cu at (189.2, 52.7)
- added C9: C, Resistors_SMD:R_0805_HandSoldering, F.Cu at (109.5, 34.0)
- added J10: Conn_01x01, TuftsRacing2018:MountingPadM3, F.Cu at (3.56, 16.3)
- added J11: Conn_01x01, TuftsRacing2018:MountingPadM3, F.Cu at (199.6, 85.3)
- added J12: Conn_01x01, TuftsRacing2018:MountingPadM3, F.Cu at (199.6, 16.3)
- added J9: Conn_01x01, TuftsRacing2018:MountingPadM3, F.Cu at (3.56, 85.3)
- added R11: 10k, Resistors_SMD:R_0805_HandSoldering, F.Cu at (53.5, 57.9)
- added SW2: SW_SPDT, TO_SOT_Packages_THT:TO-220-3_Vertical, F.Cu at (84.8, 27.4)
- added Y1: Crystal, Crystals:Crystal_SMD_HC49-SD_HandSoldering, F.Cu at (161.7, 58.4)
- C1, C2, C3, C4, C5, C6: footprint Capacitors_SMD:C_0603_HandSoldering -> Resistors_SMD:R_0805_HandSoldering
- C7, C8: value CP -> C; footprint Capacitors_THT:CP_Radial_D8.0mm_P5.00mm -> Capacitors_SMD:C_0805_HandSoldering
- Q1, Q2, Q3, Q4: value Q_NMOS_DGS -> Q_NMOS_GDS; footprint TO_SOT_Packages_SMD:TO-263-2 -> TO_SOT_Packages_SMD:TO-252-2
- R1, R10, R2, R4, R5, R6, R7, R8, R9: footprint Resistors_SMD:R_0603_HandSoldering -> Resistors_SMD:R_0805_HandSoldering
- U3: footprint Housings_DIP:DIP-14_W8.89mm_SMDSocket_LongPads -> Housings_DIP:DIP-16_W8.89mm_SMDSocket_LongPads
- moved R2 187.8 mm to (22.4, 57.6)
- moved R1 180.3 mm to (10.7, 57.7), turned to 180 degrees
- moved R7 122.4 mm to (125.5, 29.8), turned to 90 degrees
- moved R8 118.5 mm to (141.7, 33.0), turned to 90 degrees
- moved C8 114.3 mm to (122.6, 34.9), turned to 270 degrees
- moved C7 111.9 mm to (125.5, 34.9), turned to 270 degrees
- moved U1 106.2 mm to (112.0, 30.5)
- moved C1 99.3 mm to (141.6, 25.4)
- moved U6 97.5 mm to (133.6, 31.4)
- moved F11 95.4 mm to (114.7, 63.1), turned to 180 degrees
- moved F10 89.1 mm to (114.7, 54.0), turned to 180 degrees
- moved F3 85.1 mm to (9.81, 50.9)
- moved F4 84.9 mm to (9.81, 33.4)
- moved F6 84.7 mm to (22.9, 50.9)
- moved F1 84.6 mm to (114.7, 45.1), turned to 180 degrees
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Connections:
- C8 pad 1: Net-(C8-Pad1) -> Net-(C7-Pad1)
- J4 pad 14: Net-(J4-Pad14) -> /CHARGER_SD
- Q1 pad 1: /RTDS- -> /Logic/RTDS
- Q1 pad 2: /Logic/RTDS -> /RTDS-
- Q2 pad 1: /BATT_FAN- -> /FAN_PWM
- Q2 pad 2: /FAN_PWM -> /BATT_FAN-
- Q3 pad 1: Net-(D2-Pad2) -> /ShutdownCircuit/IMD_FLT_5V_L
- Q3 pad 2: /ShutdownCircuit/IMD_FLT_5V_L -> Net-(D2-Pad2)
- Q4 pad 1: Net-(D4-Pad2) -> /ShutdownCircuit/BMS_FLT_5V_L
- Q4 pad 2: /ShutdownCircuit/BMS_FLT_5V_L -> Net-(D4-Pad2)
- R3 pad 1: +12V -> /ShutdownCircuit/IMD_FLT_5V_L
- R3 pad 2: /BMS_FLT -> GND
- R8 pad 1: Net-(C8-Pad1) -> Net-(C13-Pad1)
- U6 pad 9: Net-(C8-Pad1) -> Net-(C13-Pad1)
Routing:
- net /Logic/RTDS: track 0.00 -> 195.5 mm, vias 0 -> 14
- net /CONTACT_REQ: track 0.00 -> 149.3 mm, vias 0 -> 2
- net /TSMS: track 0.00 -> 138.1 mm, vias 0 -> 5
- net /SOC: track 0.00 -> 134.4 mm, vias 0 -> 2
- net /BRK_SW: track 0.00 -> 133.9 mm
- net /CHARGER_SD: track 0.00 -> 129.3 mm, vias 0 -> 4
- net /ShutdownCircuit/BMS_FLT_5V_L: track 0.00 -> 110.0 mm, vias 0 -> 6
- net /IMD_FLT_12V_LED_H: track 0.00 -> 107.4 mm
- net /SignalDelay/A1: track 0.00 -> 102.2 mm
- net /BOTS: track 30.4 -> 131.2 mm, vias 0 -> 3
- net /SignalDelay/A2: track 0.00 -> 100.6 mm
- net +5V: track 3.31 -> 103.7 mm, vias 0 -> 10
- net /BMS_FLT: track 3.09 -> 100.6 mm, vias 0 -> 3
- net /ShutdownCircuit/IMD_FLT_5V_L: track 0.00 -> 88.0 mm, vias 0 -> 6
- net GND: track 13.3 -> 92.9 mm, vias 16 -> 17
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Other:
- board outline added: 203.2 x 76.2 mm
- rule trace_min: 0.2 -> 0.1524
- rule via_min_drill: 0.3 -> 0.1524
- rule via_min_size: 0.4 -> 0.3048
- board text removed: "BMS Bullshit"

Commit message: final design competition 2018
Connections:
- J5 pad 12: Net-(J5-Pad12) -> /COCKPIT_SW
- U4 pad 14: /Logic/SECON_FWD -> /Logic/SEVCON_FWD
Routing:
- net /COCKPIT_SW: track 0.00 -> 129.0 mm, vias 0 -> 1
- net /Logic/SEVCON_FWD: track 0.00 -> 64.3 mm, vias 0 -> 2
- net +5V: track 103.7 -> 94.2 mm, vias 10 -> 9
- net /SEVCON_FLT: track 36.0 -> 36.8 mm
- net /BOTS: track 131.2 -> 130.5 mm
Other:
- board text added: "Tufts Racing 2018 - MB REV 0 Zachary Faber Manning"
